File: _saved_glass-break.sch (KiCad schematic (older format))
At the start: 10 parts, among them IC1 ATMEGA328-P, U2? admp401

Commit message: schematic update
Parts:
- R?: footprint (none) -> ~
Changed lines of the file:
@@
 F 0 "R?" V 7430 2700 50  0000 C CNN
 F 1 "1M" V 7350 2700 50  0000 C CNN
-F 2 "" V 7280 2700 50  0000 C CNN
+F 2 "~" V 7280 2700 50  0000 C CNN
 F 3 "" H 7350 2700 50  0000 C CNN
 	1    7350 2700
