File: hardware/_autosave-glass-break.kicad_pcb (KiCad board)
At the start: 2 copper layers, 90 x 57 mm, 25 parts, among them P1 USB_OTG, U11 SPX3819

Commit message: layout update
Other:
- board outline removed
Changed lines of the file:
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@@
     (links 47)
     (no_connects 30)
-    (area 0 0 0 0)
+    (area 113.924999 32.924999 204.075001 129.878601)
     (thickness 1.6)
-    (drawings 6)
+    (drawings 13)
     (tracks 0)
     (zones 0)
@@
     )
   )
-  (gr_line (start 133 87) (end 133 54.5) (angle 90) (layer Edge.Cuts) (width 0.15))
-  (gr_circle (center 133 80) (end 140 80) (layer Edge.Cuts) (width 0.15))
-  (gr_line (start 114 33) (end 114 90) (angle 90) (layer Edge.Cuts) (width 0.15))
-  (gr_line (start 204 33) (end 114 33) (angle 90) (layer Edge.Cuts) (width 0.15))
-  (gr_line (start 204 90) (end 204 33) (angle 90) (layer Edge.Cuts) (width 0.15))
-  (gr_line (start 114 90) (end 204 90) (angle 90) (layer Edge.Cuts) (width 0.15))
+  (gr_circle (center 152.5 87.5) (end 152.5 84) (layer Margin) (width 0.2))
+  (gr_line (start 193 82.5) (end 193 94.5) (angle 90) (layer Margin) (width 0.2))
+  (gr_line (start 193 82.5) (end 205 82.5) (angle 90) (layer Margin) (width 0.2))
+  (gr_line (start 193 56.5) (end 193 44.5) (angle 90) (layer Margin) (width 0.2))
+  (gr_line (start 205 56.5) (end 193 56.5) (angle 90) (layer Margin) (width 0.2))
+  (gr_line (start 132.5 56.5) (end 132.5 44.5) (angle 90) (layer Margin) (width 0.2))
+  (gr_line (start 120.5 56.5) (end 132.5 56.5) (angle 90) (layer Margin) (width 0.2))
+  (gr_line (start 132.5 82.5) (end 120.5 82.5) (angle 90) (layer Margin) (width 0.2))
+  (gr_line (start 132.5 94.5) (end 132.5 82.5) (angle 90) (layer Margin) (width 0.2))
+  (gr_line (start 120.5 44.5) (end 120.5 94.5) (angle 90) (layer Margin) (width 0.2))
+  (gr_line (start 205 44.5) (end 120.5 44.5) (angle 90) (layer Margin) (width 0.2))
+  (gr_line (start 205 94.5) (end 205 44.5) (angle 90) (layer Margin) (width 0.2))
+  (gr_line (start 120.5 94.5) (end 205 94.5) (angle 90) (layer Margin) (width 0.2))
 )
