File: hardware/glass-break.sch (KiCad schematic (older format))
At the start: 10 parts, among them IC1 ATMEGA328-P, U2? admp401

Commit message: update
Parts:
- removed C1: 4.7 uF, symbol C
- removed C2: 1.0uF, symbol C
- removed C3: 10pF, symbol C
- removed R1, R2: 1.5K, symbol R
- removed R4: 100K, symbol R
- removed R?: 1M, ~, symbol R
- removed U2?: admp401, symbol admp401
- removed U?: OP275, symbol OP275
- added C?: 100nF, symbol C
- added C? (x2): 10uF, symbol C
- added Q? (x2): BFR92, SOT-323, symbol BFR92
- added R? (x2): 10K, symbol R
- added R? (x2): 1K, symbol R
- added R?: 4.7K, symbol R
Connections:
- net labels added: +5V
- wire segments 29 -> 28

Commit message: update
Parts:
- removed IC1: ATMEGA328-P, DIL28, symbol ATMEGA328-P
- added C?: 10UF, symbol C
- added D? (x2), red: D, symbol D
- added JP1: CONN_01X06, symbol CONN_01X06
- added JP4, JP5: CONN_01X10, symbol CONN_01X10
- added MBR120 (x2): ZENER, symbol ZENER
- added R3, R? (x4): 10K, symbol R
- added R?: 1k, symbol R
- added SW? (x2): SW_PUSH, symbol SW_PUSH
- added U1?: SPX3819, symbol SPX3819
- added U?: esp12, symbol esp12
Connections:
- net labels added: +3.3V, +BATT, 3.3V, ADC, CH_PD, GPIO0, GPIO12, GPIO13, GPIO14, GPIO15, GPIO16, GPIO2, GPIO4, GPIO5, LDO_EN, RESET, RESET_5V, RXD, RXD_5V, TXD, VBAT, VIN
- net labels removed: VCC
- wire segments 28 -> 80
Other:
- moved on the sheet: C?, Q?, R?

Commit message: update
Parts:
- removed C?: 100nF, symbol C
- removed C? (x2): 10uF, symbol C
- removed Q? (x2): BFR92, SOT-323, symbol BFR92
- removed R? (x2): 10K, symbol R
- removed R? (x2): 1K, symbol R
- removed R?: 4.7K, symbol R
- added C? (x3): C, symbol C
- added P?: USB_OTG, symbol USB_OTG
- added R? (x4): R, symbol R
- added U?: admp401, symbol admp401
- added U?: OP275, symbol OP275
Connections:
- net labels added: VCC
- net labels removed: +5V
- wire segments 80 -> 82
Other:
- moved on the sheet: U?

Commit message: sch update
Parts:
- added R11: 1k, symbol R
- added red2: D, symbol D
- gave numbers to parts that had none: 22
- renumbered red to red1
Connections:
- wire segments 82 -> 85

Commit message: update
Parts:
- removed R1, R11: 1k, symbol R
- removed R4, R5, R6: 10K, symbol R
- removed R8: R, symbol R
- removed SW1, SW2: SW_PUSH, symbol SW_PUSH
- removed U3: admp401, symbol admp401
- removed red1, red2: D, symbol D
- added D? (x2): LED, symbol LED
- added JP?: CONN_01X10, symbol CONN_01X10
- added R? (x5): 10K, symbol R
- added R?: 1K, symbol R
- added R?: 2.2K, symbol R
- added SW? (x3): SW_PUSH, symbol SW_PUSH
- added U?: electret_microphone, symbol electret_microphone
- C2: value C -> 12pF
- C3: value C -> 1uF
- C4: value C -> 4.7 uF
- R10: value R -> 10K
- R2: value 10K -> 1K
- R7: value R -> 1M
- R9: value R -> 10k
Connections:
- net labels added: LD0_EN
- net labels removed: VBAT, VCC
- wire segments 85 -> 104
Other:
- moved on the sheet: C1, C2, C3, C4, D1, D2, JP1, JP4, JP5, MBR120, P1, R10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

Commit message: update
Parts:
- C2, C3, C4: footprint (none) -> Capacitors_SMD:C_0805
- D1, D2, D? (x2): footprint (none) -> LEDs:LED_0805
- R10, R2, R3, R7, R9, R? (x7): footprint (none) -> Resistors_SMD:R_0805
Changed lines of the file:
@@
 F 0 "R3" V 2180 5800 50  0000 C CNN
 F 1 "10K" V 2100 5800 50  0000 C CNN
-F 2 "" V 2030 5800 50  0000 C CNN
+F 2 "Resistors_SMD:R_0805" V 2030 5800 50  0000 C CNN
 F 3 "" H 2100 5800 50  0000 C CNN
 	1    2100 5800
@@
 F 0 "D1" H 2500 4200 50  0000 C CNN
 F 1 "D" H 2500 4000 50  0000 C CNN
-F 2 "" H 2500 4100 50  0000 C CNN
+F 2 "LEDs:LED_0805" H 2500 4100 50  0000 C CNN
 F 3 "" H 2500 4100 50  0000 C CNN
 	1    2500 4100
@@
 F 0 "D2" H 2500 4300 50  0000 C CNN
 F 1 "D" H 2500 4100 50  0000 C CNN
-F 2 "" H 2500 4200 50  0000 C CNN
+F 2 "LEDs:LED_0805" H 2500 4200 50  0000 C CNN
 F 3 "" H 2500 4200 50  0000 C CNN
 	1    2500 4200
@@
 F 0 "C3" H 6575 2400 50  0000 L CNN
 F 1 "1uF" H 6575 2200 50  0000 L CNN
-F 2 "" H 6588 2150 50  0000 C CNN
+F 2 "Capacitors_SMD:C_0805" H 6588 2150 50  0000 C CNN
 F 3 "" H 6550 2300 50  0000 C CNN
 	1    6550 2300
@@
 F 0 "C2" H 7525 950 50  0000 L CNN
 F 1 "12pF" H 7525 750 50  0000 L CNN
-F 2 "" H 7538 700 50  0000 C CNN
+F 2 "Capacitors_SMD:C_0805" H 7538 700 50  0000 C CNN
 F 3 "" H 7500 850 50  0000 C CNN
 	1    7500 850
@@
 F 0 "C4" H 6275 1950 50  0000 L CNN
 F 1 "4.7 uF" H 6275 1750 50  0000 L CNN
-F 2 "" H 6288 1700 50  0000 C CNN
+F 2 "Capacitors_SMD:C_0805" H 6288 1700 50  0000 C CNN
 F 3 "" H 6250 1850 50  0000 C CNN
 	1    6250 1850
@@
 F 0 "R7" V 7580 1050 50  0000 C CNN
 F 1 "1M" V 7500 1050 50  0000 C CNN
-F 2 "" V 7430 1050 50  0000 C CNN
+F 2 "Resistors_SMD:R_0805" V 7430 1050 50  0000 C CNN
 F 3 "" H 7500 1050 50  0000 C CNN
 	1    7500 1050
@@
 F 0 "R9" V 6980 2300 50  0000 C CNN
 F 1 "10k" V 6900 2300 50  0000 C CNN
-F 2 "" V 6830 2300 50  0000 C CNN
+F 2 "Resistors_SMD:R_0805" V 6830 2300 50  0000 C CNN
 F 3 "" H 6900 2300 50  0000 C CNN
 	1    6900 2300
@@
 F 0 "R10" V 6730 1850 50  0000 C CNN
 F 1 "10K" V 6650 1850 50  0000 C CNN
-F 2 "" V 6580 1850 50  0000 C CNN
+F 2 "Resistors_SMD:R_0805" V 6580 1850 50  0000 C CNN
 F 3 "" H 6650 1850 50  0000 C CNN
 	1    6650 1850
@@
 F 0 "R2" V 1180 2100 50  0000 C CNN
 F 1 "1K" V 1100 2100 50  0000 C CNN
-F 2 "" V 1030 2100 50  0000 C CNN
+F 2 "Resistors_SMD:R_0805" V 1030 2100 50  0000 C CNN
 F 3 "" H 1100 2100 50  0000 C CNN
 	1    1100 2100
@@
 F 0 "R?" V 1980 1450 50  0000 C CNN
 F 1 "10K" V 1900 1450 50  0000 C CNN
-F 2 "" V 1830 1450 50  0000 C CNN
+F 2 "Resistors_SMD:R_0805" V 1830 1450 50  0000 C CNN
 F 3 "" H 1900 1450 50  0000 C CNN
 	1    1900 1450
@@
 F 0 "R?" V 2330 2200 50  0000 C CNN
 F 1 "10K" V 2250 2200 50  0000 C CNN
-F 2 "" V 2180 2200 50  0000 C CNN
+F 2 "Resistors_SMD:R_0805" V 2180 2200 50  0000 C CNN
 F 3 "" H 2250 2200 50  0000 C CNN
 	1    2250 2200
@@
 F 0 "R?" V 2730 2200 50  0000 C CNN
 F 1 "10K" V 2650 2200 50  0000 C CNN
-F 2 "" V 2580 2200 50  0000 C CNN
+F 2 "Resistors_SMD:R_0805" V 2580 2200 50  0000 C CNN
 F 3 "" H 2650 2200 50  0000 C CNN
 	1    2650 2200
@@
 F 0 "R?" V 3130 2200 50  0000 C CNN
 F 1 "10K" V 3050 2200 50  0000 C CNN
-F 2 "" V 2980 2200 50  0000 C CNN
+F 2 "Resistors_SMD:R_0805" V 2980 2200 50  0000 C CNN
 F 3 "" H 3050 2200 50  0000 C CNN
 	1    3050 2200
@@
 F 0 "D?" H 1100 1700 50  0000 C CNN
 F 1 "LED" H 1100 1500 50  0000 C CNN
-F 2 "" H 1100 1600 50  0000 C CNN
+F 2 "LEDs:LED_0805" H 1100 1600 50  0000 C CNN
 F 3 "" H 1100 1600 50  0000 C CNN
 	1    1100 1600
@@
 F 0 "R?" V 3380 2150 50  0000 C CNN
 F 1 "1K" V 3300 2150 50  0000 C CNN
-F 2 "" V 3230 2150 50  0000 C CNN
+F 2 "Resistors_SMD:R_0805" V 3230 2150 50  0000 C CNN
 F 3 "" H 3300 2150 50  0000 C CNN
 	1    3300 2150
@@
 F 0 "D?" H 3300 1750 50  0000 C CNN
 F 1 "LED" H 3300 1550 50  0000 C CNN
-F 2 "" H 3300 1650 50  0000 C CNN
+F 2 "LEDs:LED_0805" H 3300 1650 50  0000 C CNN
 F 3 "" H 3300 1650 50  0000 C CNN
 	1    3300 1650
@@
 F 0 "R?" V 6980 1600 50  0000 C CNN
 F 1 "10K" V 6900 1600 50  0000 C CNN
-F 2 "" V 6830 1600 50  0000 C CNN
+F 2 "Resistors_SMD:R_0805" V 6830 1600 50  0000 C CNN
 F 3 "" H 6900 1600 50  0000 C CNN
 	1    6900 1600
@@
 F 0 "R?" V 6080 1500 50  0000 C CNN
 F 1 "2.2K" V 6000 1500 50  0000 C CNN
-F 2 "" V 5930 1500 50  0000 C CNN
+F 2 "Resistors_SMD:R_0805" V 5930 1500 50  0000 C CNN
 F 3 "" H 6000 1500 50  0000 C CNN
 	1    6000 1500

Commit message: update
Parts:
- removed JP?: CONN_01X10, symbol CONN_01X10
- C1: footprint (none) -> Capacitors_SMD:C_0805
- JP1: footprint (none) -> Pin_Headers:Pin_Header_Angled_1x06
- JP4, JP5: footprint (none) -> Pin_Headers:Pin_Header_Angled_1x10
- P1: footprint (none) -> Connect:USB_Micro-B
- U11: footprint (none) -> TO_SOT_Packages_SMD:SC-70-5
- gave numbers to parts that had none: 13

Commit message: layout update
Parts:
- renumbered MBR120 to MBR120-1, MBR120 to MBR120-2
Other:
- moved on the sheet: MBR120-2
