File: hardware/glass-break.sch (KiCad schematic (older format))
At the start: 33 parts, among them P1 USB_OTG, SW1 SW_PUSH, SW2 SW_PUSH, SW3 SW_PUSH, U1 esp12, U11 SPX3819, U2 OP275, U3 electret_microphone

Commit message: update
Parts:
- JP1: footprint Pin_Headers:Pin_Header_Angled_1x06 -> Pin_Headers:Pin_Header_Straight_1x06
- JP4, JP5: footprint Pin_Headers:Pin_Header_Angled_1x10 -> Pin_Headers:Pin_Header_Straight_1x10
- renumbered MBR120-2 to MBR120, MBR120-1 to MBR120
Other:
- moved on the sheet: MBR120

Commit message: datasheetupdate
Parts:
- C1: value 10UF -> 1uf
- U11: footprint TO_SOT_Packages_SMD:SC-70-5 -> TO_SOT_Packages_SMD:SOT-23-5
- renumbered MBR120 to MBR120-1, MBR120 to MBR120-2
Changed lines of the file:
@@
 F 1 "esp12" V 9150 1950 60  0000 C CNN
 F 2 "" H 9200 2400 60  0000 C CNN
-F 3 "" H 9200 2400 60  0000 C CNN
+F 3 "http://www.mouser.com/pdfdocs/adafruithuzzahesp8266breakout.PDF" H 9200 2400 60  0001 C CNN
 	1    9150 2050
 	1    0    0    -1
@@
 F 0 "U11" H 3150 5900 50  0000 C CNN
 F 1 "SPX3819" H 3550 5900 50  0000 C CNN
-F 2 "TO_SOT_Packages_SMD:SC-70-5" H 3400 5150 50  0000 C CIN
-F 3 "" H 3450 5050 50  0001 C CNN
+F 2 "TO_SOT_Packages_SMD:SOT-23-5" H 3400 5150 50  0000 C CIN
+F 3 "http://www.mouser.com/ds/2/146/SPX3819_DS_R200_082312-17072.pdf" H 3450 5050 50  0001 C CNN
 	1    3400 5550
 	1    0    0    -1
@@
 F 1 "10K" V 2100 5800 50  0000 C CNN
 F 2 "Resistors_SMD:R_0805" V 2030 5800 50  0000 C CNN
-F 3 "" H 2100 5800 50  0000 C CNN
+F 3 "http://www.mouser.com/ds/2/315/AOA0000CE2-37512.pdf" H 2100 5800 50  0001 C CNN
 	1    2100 5800
 	1    0    0    -1
@@
 P 1750 5800
 F 0 "C1" H 1775 5900 50  0000 L CNN
-F 1 "10UF" H 1775 5700 50  0000 L CNN
+F 1 "1uf" H 1775 5700 50  0000 L CNN
 F 2 "Capacitors_SMD:C_0805" V 1788 5650 50  0000 C CNN
 F 3 "" H 1750 5800 50  0000 C CNN
@@
 $EndComp
 $Comp
-L ZENER MBR120
+L ZENER MBR120-2
 U 1 1 56C66052
 P 2100 5000
-F 0 "MBR120" H 2100 5100 50  0000 C CNN
+F 0 "MBR120-2" H 2100 5100 50  0000 C CNN
 F 1 "ZENER" H 2100 4900 50  0000 C CNN
 F 2 "" H 2100 5000 50  0000 C CNN
@@
 $EndComp
 $Comp
-L ZENER MBR120
+L ZENER MBR120-1
 U 1 1 56C660C8
 P 1750 5000
-F 0 "MBR120" H 1750 5100 50  0000 C CNN
+F 0 "MBR120-1" H 1750 5100 50  0000 C CNN
 F 1 "ZENER" H 1750 4900 50  0000 C CNN
 F 2 "" H 1750 5000 50  0000 C CNN
@@
 F 1 "1uF" H 6575 2200 50  0000 L CNN
 F 2 "Capacitors_SMD:C_0805" H 6588 2150 50  0000 C CNN
-F 3 "" H 6550 2300 50  0000 C CNN
+F 3 "http://www.mouser.com/ds/2/400/lcc_commercial_general_en-837201.pdf" H 6550 2300 50  0001 C CNN
 	1    6550 2300
 	-1   0    0    -1
@@
 F 1 "12pF" H 7525 750 50  0000 L CNN
 F 2 "Capacitors_SMD:C_0805" H 7538 700 50  0000 C CNN
-F 3 "" H 7500 850 50  0000 C CNN
+F 3 "http://www.mouser.com/ds/2/40/C0GNP0-Dielectric-775593.pdf" H 7500 850 50  0001 C CNN
 	1    7500 850
 	0    1    -1   0
@@
 F 1 "4.7 uF" H 6275 1750 50  0000 L CNN
 F 2 "Capacitors_SMD:C_0805" H 6288 1700 50  0000 C CNN
-F 3 "" H 6250 1850 50  0000 C CNN
+F 3 "http://www.mouser.com/ds/2/212/KEM_C1006_X5R_SMD-348855.pdf" H 6250 1850 50  0001 C CNN
 	1    6250 1850
 	0    1    -1   0
@@
 F 1 "1M" V 7500 1050 50  0000 C CNN
 F 2 "Resistors_SMD:R_0805" V 7430 1050 50  0000 C CNN
-F 3 "" H 7500 1050 50  0000 C CNN
+F 3 "http://www.mouser.com/ds/2/315/AOA0000CE1-37422.pdf" H 7500 1050 50  0001 C CNN
 	1    7500 1050
 	0    -1   1    0
@@
 F 1 "10k" V 6900 2300 50  0000 C CNN
 F 2 "Resistors_SMD:R_0805" V 6830 2300 50  0000 C CNN
-F 3 "" H 6900 2300 50  0000 C CNN
+F 3 "http://www.mouser.com/ds/2/315/AOA0000CE2-37512.pdf" H 6900 2300 50  0001 C CNN
 	1    6900 2300
 	-1   0    0    -1
@@
 F 1 "10K" V 6650 1850 50  0000 C CNN
 F 2 "Resistors_SMD:R_0805" V 6580 1850 50  0000 C CNN
-F 3 "" H 6650 1850 50  0000 C CNN
+F 3 "http://www.mouser.com/ds/2/315/AOA0000CE2-37512.pdf" H 6650 1850 50  0001 C CNN
 	1    6650 1850
 	0    -1   1    0
@@
 F 1 "10K" V 2250 2200 50  0000 C CNN
 F 2 "Resistors_SMD:R_0805" V 2180 2200 50  0000 C CNN
-F 3 "" H 2250 2200 50  0000 C CNN
+F 3 "http://www.mouser.com/ds/2/315/AOA0000CE2-37512.pdf" H 2250 2200 50  0001 C CNN
 	1    2250 2200
 	1    0    0    -1
@@
 F 1 "10K" V 2650 2200 50  0000 C CNN
 F 2 "Resistors_SMD:R_0805" V 2580 2200 50  0000 C CNN
-F 3 "" H 2650 2200 50  0000 C CNN
+F 3 "http://www.mouser.com/ds/2/315/AOA0000CE2-37512.pdf" H 2650 2200 50  0001 C CNN
 	1    2650 2200
 	1    0    0    -1
@@
 F 1 "10K" V 3050 2200 50  0000 C CNN
 F 2 "Resistors_SMD:R_0805" V 2980 2200 50  0000 C CNN
-F 3 "" H 3050 2200 50  0000 C CNN
+F 3 "http://www.mouser.com/ds/2/315/AOA0000CE2-37512.pdf" H 3050 2200 50  0001 C CNN
 	1    3050 2200
 	1    0    0    -1
@@
 F 1 "1K" V 3300 2150 50  0000 C CNN
 F 2 "Resistors_SMD:R_0805" V 3230 2150 50  0000 C CNN
-F 3 "" H 3300 2150 50  0000 C CNN
+F 3 "http://www.mouser.com/ds/2/315/AOA0000CE2-37512.pdf" H 3300 2150 50  0001 C CNN
 	1    3300 2150
 	1    0    0    -1
@@
 F 1 "10K" V 6900 1600 50  0000 C CNN
 F 2 "Resistors_SMD:R_0805" V 6830 1600 50  0000 C CNN
-F 3 "" H 6900 1600 50  0000 C CNN
+F 3 "http://www.mouser.com/ds/2/315/AOA0000CE2-37512.pdf" H 6900 1600 50  0001 C CNN
 	1    6900 1600
 	-1   0    0    -1
@@
 F 1 "2.2K" V 6000 1500 50  0000 C CNN
 F 2 "Resistors_SMD:R_0805" V 5930 1500 50  0000 C CNN
-F 3 "" H 6000 1500 50  0000 C CNN
+F 3 "http://www.mouser.com/ds/2/315/AOA0000CE1-37422.pdf" H 6000 1500 50  0001 C CNN
 	1    6000 1500
 	-1   0    0    -1

Commit message: footprint update
Parts:
- C3: value 1uF -> 10uF
- MBR120-1, MBR120-2: footprint (none) -> Diodes_SMD:SOD-123
- SW1, SW2, SW3: footprint (none) -> Buttons_Switches_SMD:SW_SPST_KMR2
- U1: footprint (none) -> esp12e:Esp12e
- U2: footprint (none) -> Housings_SOIC:SOIC-8_3.9x4.9mm_Pitch1.27mm
- U3: footprint (none) -> esp12e:Electret
Connections:
- net GND: no longer JP1.4 (P4), JP4.8 (P8), MBR120-1.2 (A)
- new net +5V: JP1.4 (P4), JP4.8 (P8), MBR120-1.2 (A)

Commit message: pcd update
Parts:
- U11: footprint TO_SOT_Packages_SMD:SOT-23-5 -> esp12e:SOT-23-5(MOD)
Connections:
- net +5V: now also P1.1 (VCC)
- net GND: no longer P1.1 (VCC)
- net LD0_EN: no longer R3.2, U11.3 (GND)
- net RESET: now also U1.1 (RESET)
- net RESET_5V: no longer U1.1 (RESET)
- net RXD: no longer D2.1 (K), JP1.3 (P3), JP5.9 (P9)
- new net: R3.2, U11.3 (GND)
- new net RXD_5V: D2.1 (K), JP1.3 (P3), JP5.9 (P9)
Changed lines of the file:
@@
 F 1 "esp12" V 9150 1950 60  0000 C CNN
 F 2 "esp12e:Esp12e" H 9200 2400 60  0000 C CNN
-F 3 "http://www.mouser.com/ProductDetail/Adafruit/2491/?qs=sGAEpiMZZMsMyYRRhGMFNh3isolDxGLO%2fZK71n5k6Ow%3d" H 9200 2400 60  0001 C CNN
+F 3 "https://learn.adafruit.com/adafruit-huzzah-esp8266-breakout?view=all" H 9200 2400 60  0001 C CNN
 	1    9150 2050
 	1    0    0    -1
@@
 F 0 "U11" H 3150 5900 50  0000 C CNN
 F 1 "SPX3819" H 3550 5900 50  0000 C CNN
-F 2 "TO_SOT_Packages_SMD:SOT-23-5" H 3400 5150 50  0000 C CIN
+F 2 "esp12e:SOT-23-5(MOD)" H 3400 5150 50  0000 C CIN
 F 3 "http://www.mouser.com/ds/2/146/SPX3819_DS_R200_082312-17072.pdf" H 3450 5050 50  0001 C CNN
 	1    3400 5550
@@
 F 1 "ZENER" H 2100 4900 50  0000 C CNN
 F 2 "Diodes_SMD:SOD-123" H 2100 5000 50  0000 C CNN
-F 3 "http://www.mouser.com/ds/2/308/MBR120VLSFT1-D-107081.pdf" H 2100 5000 50  0000 C CNN
+F 3 "http://www.mouser.com/ds/2/308/MBR120VLSFT1-D-107081.pdf" H 2100 5000 50  0001 C CNN
 	1    2100 5000
 	0    -1   -1   0
@@
 F 1 "ZENER" H 1750 4900 50  0000 C CNN
 F 2 "Diodes_SMD:SOD-123" H 1750 5000 50  0000 C CNN
-F 3 "http://www.mouser.com/ds/2/308/MBR120VLSFT1-D-107081.pdf" H 1750 5000 50  0000 C CNN
+F 3 "http://www.mouser.com/ds/2/308/MBR120VLSFT1-D-107081.pdf" H 1750 5000 50  0001 C CNN
 	1    1750 5000
 	0    -1   -1   0
@@
 	1    0    0    -1
 $EndComp
-Text Label 2750 5550 2    39   ~ 0
-LDO_EN
 $Comp
 L D D1
@@
 RESET
 Text GLabel 1950 4200 0    60   Input ~ 0
-RXD
+RXD_5V
 Text GLabel 1950 4100 0    60   Input ~ 0
 RESET_5V
@@
 Wire Wire Line
 	5400 1850 6100 1850
-Wire Wire Line
-	7950 5150 7950 4950
 Wire Wire Line
 	8350 4950 8350 5150
@@
 GPIO15
 Text GLabel 10200 1950 2    60   Input ~ 0
-RXD_5V
+RXD
 Text GLabel 10200 1850 2    60   Input ~ 0
 TXD
@@
 RESET_5V
 Text GLabel 8500 1350 1    60   Input ~ 0
-RESET_5V
-Text GLabel 8500 1350 1    60   Input ~ 0
-RESET_5V
-Text GLabel 8500 1350 1    60   Input ~ 0
-RESET_5V
-Text GLabel 8500 1350 1    60   Input ~ 0
-RESET_5V
+RESET
 Wire Wire Line
 	8500 1350 8500 1850
@@
 	8300 2450 8500 2450
 $Comp
-L VIN #PWR027
-U 1 1 56DA93CD
-P 7950 5150
-F 0 "#PWR027" H 7950 4900 50  0001 C CNN
-F 1 "VIN" H 7950 5000 50  0000 C CNN
-F 2 "" H 7950 5150 50  0000 C CNN
-F 3 "" H 7950 5150 50  0000 C CNN
-	1    7950 5150
-	1    0    0    -1
-$EndComp
-$Comp
 L R R12
 U 1 1 56DAB83F
@@
 	6000 1350 6000 1250
 $Comp
-L +3.3V #PWR028
+L +3.3V #PWR027
 U 1 1 56DABCDE
 P 6000 1250
-F 0 "#PWR028" H 6000 1100 50  0001 C CNN
+F 0 "#PWR027" H 6000 1100 50  0001 C CNN
 F 1 "+3.3V" H 6000 1390 50  0000 C CNN
 F 2 "" H 6000 1250 50  0000 C CNN
@@
 	5550 2150 5550 2250
 $Comp
-L +5V #PWR029
+L +5V #PWR028
 U 1 1 56DE3201
 P 7650 4000
-F 0 "#PWR029" H 7650 3850 50  0001 C CNN
+F 0 "#PWR028" H 7650 3850 50  0001 C CNN
 F 1 "+5V" H 7650 4140 50  0000 C CNN
 F 2 "" H 7650 4000 50  0000 C CNN
@@
 	8550 4000 7650 4000
 $Comp
-L +5V #PWR030
+L +5V #PWR029
 U 1 1 56DE3BD1
 P 1750 4700
-F 0 "#PWR030" H 1750 4550 50  0001 C CNN
+F 0 "#PWR029" H 1750 4550 50  0001 C CNN
 F 1 "+5V" H 1750 4840 50  0000 C CNN
 F 2 "" H 1750 4700 50  0000 C CNN
@@
 $EndComp
 $Comp
-L +5V #PWR031
+L +5V #PWR030
 U 1 1 56DE3BF8
 P 9200 5050
-F 0 "#PWR031" H 9200 4900 50  0001 C CNN
+F 0 "#PWR030" H 9200 4900 50  0001 C CNN
 F 1 "+5V" H 9200 5190 50  0000 C CNN
 F 2 "" H 9200 5050 50  0000 C CNN
@@
 Wire Wire Line
 	9200 4750 9200 5050
+$Comp
+L +5V #PWR031
+U 1 1 56DEFE2B
+P 7950 5150
+F 0 "#PWR031" H 7950 5000 50  0001 C CNN
+F 1 "+5V" H 7950 5290 50  0000 C CNN
+F 2 "" H 7950 5150 50  0000 C CNN
+F 3 "" H 7950 5150 50  0000 C CNN
+	1    7950 5150
+	-1   0    0    1
+$EndComp
+Wire Wire Line
+	7950 5150 7950 4950
 $EndSCHEMATC

Commit message: PCB attempt
Connections:
- net GND: now also P1.6 (shield)
Other:
- moved on the sheet: P1
Changed lines of the file:
@@
 L USB_OTG P1
 U 1 1 56C75F6C
-P 8150 4650
-F 0 "P1" H 8475 4525 50  0000 C CNN
-F 1 "USB_OTG" H 8150 4850 50  0000 C CNN
-F 2 "Connect:USB_Micro-B" H 8100 4550 50  0000 C CNN
-F 3 "" V 8100 4550 50  0000 C CNN
-	1    8150 4650
+P 1050 4600
+F 0 "P1" H 1375 4475 50  0000 C CNN
+F 1 "USB_OTG" H 1050 4800 50  0000 C CNN
+F 2 "Connect:USB_Micro-B" H 1000 4500 50  0000 C CNN
+F 3 "" V 1000 4500 50  0000 C CNN
+	1    1050 4600
 	1    0    0    -1
 $EndComp
@@
 	5400 1850 6100 1850
 Wire Wire Line
-	8350 4950 8350 5150
+	1250 4900 1250 5100
 $Comp
 L +BATT #PWR018
@@
 L GND #PWR025
 U 1 1 56DA02A1
-P 8350 5150
-F 0 "#PWR025" H 8350 4900 50  0001 C CNN
-F 1 "GND" H 8350 5000 50  0000 C CNN
-F 2 "" H 8350 5150 50  0000 C CNN
-F 3 "" H 8350 5150 50  0000 C CNN
-	1    8350 5150
+P 1250 5100
+F 0 "#PWR025" H 1250 4850 50  0001 C CNN
+F 1 "GND" H 1250 4950 50  0000 C CNN
+F 2 "" H 1250 5100 50  0000 C CNN
+F 3 "" H 1250 5100 50  0000 C CNN
+	1    1250 5100
 	1    0    0    -1
 $EndComp
@@
 L +5V #PWR031
 U 1 1 56DEFE2B
-P 7950 5150
-F 0 "#PWR031" H 7950 5000 50  0001 C CNN
-F 1 "+5V" H 7950 5290 50  0000 C CNN
-F 2 "" H 7950 5150 50  0000 C CNN
-F 3 "" H 7950 5150 50  0000 C CNN
-	1    7950 5150
+P 850 5100
+F 0 "#PWR031" H 850 4950 50  0001 C CNN
+F 1 "+5V" H 850 5240 50  0000 C CNN
+F 2 "" H 850 5100 50  0000 C CNN
+F 3 "" H 850 5100 50  0000 C CNN
+	1    850  5100
 	-1   0    0    1
 $EndComp
 Wire Wire Line
-	7950 5150 7950 4950
+	850  5100 850  4900
+Wire Wire Line
+	1450 4500 1450 4950
+Wire Wire Line
+	1450 4950 1250 4950
+Connection ~ 1250 4950
 $EndSCHEMATC

Commit message: update
Other:
- moved on the sheet: JP1, JP4, JP5

Commit message: update
Connections:
- net +3V3: no longer U1.8 (3.3V)
- net ADC: no longer U1.2 (ADC)
Other:
- moved on the sheet: U1
Changed lines of the file:
@@
 L esp12 U1
 U 1 1 56C613D6
-P 9150 2050
-F 0 "U1" H 9500 1350 60  0000 C CNN
-F 1 "esp12" V 9150 1950 60  0000 C CNN
-F 2 "esp12e:Esp12e" H 9200 2400 60  0000 C CNN
-F 3 "https://learn.adafruit.com/adafruit-huzzah-esp8266-breakout?view=all" H 9200 2400 60  0001 C CNN
-	1    9150 2050
+P 12700 2000
+F 0 "U1" H 13050 1300 60  0000 C CNN
+F 1 "esp12" V 12700 1900 60  0000 C CNN
+F 2 "esp12e:Esp12e" H 12750 2350 60  0000 C CNN
+F 3 "https://learn.adafruit.com/adafruit-huzzah-esp8266-breakout?view=all" H 12750 2350 60  0001 C CNN
+	1    12700 2000
 	1    0    0    -1
 $EndComp
@@
 F 0 "U2" H 7500 2100 50  0000 L CNN
 F 1 "OP275" H 7500 1800 50  0000 L CNN
-F 2 "Housings_SOIC:SOIC-8_3.9x4.9mm_Pitch1.27mm" H 7400 2000 50  0000 C CNN
-F 3 "http://www.mouser.com/ds/2/609/OP275-879536.pdf" H 7500 2100 50  0000 C CNN
+F 2 "Housings_SOIC:SOIC-8_3.9x4.9mm_Pitch1.27mm" H 7400 2000 50  0001 C CNN
+F 3 "http://www.mouser.com/ds/2/609/OP275-879536.pdf" H 7500 2100 50  0001 C CNN
 	1    7500 1950
 	1    0    0    1
@@
 L +3.3V #PWR30
 U 1 1 56C7E707
-P 7950 2550
-F 0 "#PWR30" H 7950 2400 50  0001 C CNN
-F 1 "+3.3V" H 7950 2690 50  0000 C CNN
-F 2 "" H 7950 2550 50  0000 C CNN
-F 3 "" H 7950 2550 50  0000 C CNN
-	1    7950 2550
+P 11650 2800
+F 0 "#PWR30" H 11650 2650 50  0001 C CNN
+F 1 "+3.3V" H 11650 2940 50  0000 C CNN
+F 2 "" H 11650 2800 50  0000 C CNN
+F 3 "" H 11650 2800 50  0000 C CNN
+	1    11650 2800
 	0    -1   1    0
 $EndComp
-Text GLabel 8250 1800 1    60   Input ~ 0
+Text GLabel 8250 1950 2    60   Input ~ 0
 ADC
 Text GLabel 5000 4000 0    60   Input ~ 0
@@
 L GND #PWR32
 U 1 1 56D896D0
-P 9950 2700
-F 0 "#PWR32" H 9950 2450 50  0001 C CNN
-F 1 "GND" H 9950 2550 50  0000 C CNN
-F 2 "" H 9950 2700 50  0000 C CNN
-F 3 "" H 9950 2700 50  0000 C CNN
-	1    9950 2700
+P 13500 2650
+F 0 "#PWR32" H 13500 2400 50  0001 C CNN
+F 1 "GND" H 13500 2500 50  0000 C CNN
+F 2 "" H 13500 2650 50  0000 C CNN
+F 3 "" H 13500 2650 50  0000 C CNN
+	1    13500 2650
 	1    0    0    -1
 $EndComp
@@
 	1    0    0    -1
 $EndComp
-Text GLabel 10200 2350 2    60   Input ~ 0
+Text GLabel 13750 2300 2    60   Input ~ 0
 GPIO2
-Text GLabel 10200 2250 2    60   Input ~ 0
+Text GLabel 13750 2200 2    60   Input ~ 0
 GPIO0
-Text GLabel 10200 2150 2    60   Input ~ 0
+Text GLabel 13750 2100 2    60   Input ~ 0
 GPIO4
-Text GLabel 10200 2050 2    60   Input ~ 0
+Text GLabel 13750 2000 2    60   Input ~ 0
 GPIO5
-Text GLabel 10200 2450 2    60   Input ~ 0
+Text GLabel 13750 2400 2    60   Input ~ 0
 GPIO15
-Text GLabel 10200 1950 2    60   Input ~ 0
+Text GLabel 13750 1900 2    60   Input ~ 0
 RXD
-Text GLabel 10200 1850 2    60   Input ~ 0
+Text GLabel 13750 1800 2    60   Input ~ 0
 TXD
 Text Label 5150 3800 0    39   ~ 0
@@
 Text GLabel 5000 3800 0    60   Input ~ 0
 RESET_5V
-Text GLabel 8500 1350 1    60   Input ~ 0
+Text GLabel 12050 1300 1    60   Input ~ 0
 RESET
-Text GLabel 8300 2250 0    60   Input ~ 0
+Text GLabel 11850 2200 0    60   Input ~ 0
 GPIO14
-Text GLabel 8300 2350 0    60   Input ~ 0
+Text GLabel 11850 2300 0    60   Input ~ 0
 GPIO12
-Text GLabel 8300 2450 0    60   Input ~ 0
+Text GLabel 11850 2400 0    60   Input ~ 0
 GPIO13
-Text GLabel 8300 2050 0    60   Input ~ 0
+Text GLabel 11850 2000 0    60   Input ~ 0
 CH_PD
-Text GLabel 8300 2150 0    60   Input ~ 0
+Text GLabel 11850 2100 0    60   Input ~ 0
 GPIO16
 $Comp
@@
 	7400 2250 7400 2500
 Wire Wire Line
-	7800 1950 8500 1950
-Wire Wire Line
-	7950 2550 8500 2550
+	11350 1900 12050 1900
+Wire Wire Line
+	11500 2500 12050 2500
 Wire Wire Line
 	6600 4200 7000 4200
@@
 	6600 4300 7000 4300
 Wire Wire Line
-	8250 1800 8250 1950
-Connection ~ 8250 1950
+	11800 1750 11800 1900
+Connection ~ 11800 1900
 Wire Wire Line
 	5000 4100 5450 4100
@@
 	3300 1450 3300 1150
 Wire Wire Line
-	9800 2550 9950 2550
-Wire Wire Line
-	9950 2550 9950 2700
+	13350 2500 13500 2500
+Wire Wire Line
+	13500 2500 13500 2650
 Wire Wire Line
 	5400 1850 6100 1850
@@
 	6300 5250 6300 5500
 Wire Wire Line
-	9800 1850 10200 1850
-Wire Wire Line
-	9800 1950 10200 1950
-Wire Wire Line
-	9800 2050 10200 2050
-Wire Wire Line
-	9800 2150 10200 2150
-Wire Wire Line
-	9800 2450 10200 2450
-Wire Wire Line
-	9800 2250 10200 2250
-Wire Wire Line
-	9800 2350 10200 2350
-Wire Wire Line
-	8500 1350 8500 1850
-Wire Wire Line
-	8300 2050 8500 2050
-Wire Wire Line
-	8300 2150 8500 2150
-Wire Wire Line
-	8300 2250 8500 2250
-Wire Wire Line
-	8300 2350 8500 2350
-Wire Wire Line
-	8300 2450 8500 2450
+	13350 1800 13750 1800
+Wire Wire Line
+	13350 1900 13750 1900
+Wire Wire Line
+	13350 2000 13750 2000
+Wire Wire Line
+	13350 2100 13750 2100
+Wire Wire Line
+	13350 2400 13750 2400
+Wire Wire Line
+	13350 2200 13750 2200
+Wire Wire Line
+	13350 2300 13750 2300
+Wire Wire Line
+	12050 1300 12050 1800
+Wire Wire Line
+	11850 2000 12050 2000
+Wire Wire Line
+	11850 2100 12050 2100
+Wire Wire Line
+	11850 2200 12050 2200
+Wire Wire Line
+	11850 2300 12050 2300
+Wire Wire Line
+	11850 2400 12050 2400
 Wire Wire Line
 	6900 1750 6900 2150
@@
 Wire Wire Line
 	1750 5950 1750 6050
+Wire Wire Line
+	7800 1950 8250 1950
 $EndSCHEMATC

Commit message: update
Parts:
- removed U1: esp12, esp12e:Esp12e, symbol esp12
- added U1: ESP-WROOM-02, garage-opener:ESP-WROOM-02, symbol ESP-WROOM-02
Connections:
- net LD0_EN is gone; now on net GND: JP5.2 (P2)
- net +3V3: now also JP4.3 (P3), U1.18 (3V3)
- net ADC: now also U1.3 (TOUT)
- net GND: now also U1.1 (GND), U1.10 (GND), U1.6 (GND)
- net GPIO0: now also U1.11 (IO0); no longer JP5.6 (P6)
- net GPIO12: now also U1.15 (IO12); no longer JP4.6 (P6)
- net GPIO13: now also U1.14 (IO13); no longer JP4.7 (P7)
- net GPIO14: now also U1.16 (IO14); no longer JP4.5 (P5)
- net GPIO15: now also U1.13 (IO15); no longer JP5.4 (P4)
- net GPIO16: now also U1.2 (IO16); no longer JP4.4 (P4)
- net GPIO2: now also U1.12 (IO2); no longer JP5.5 (P5)
- net GPIO4: now also U1.9 (IO4); no longer JP5.7 (P7)
- net GPIO5: now also U1.5 (IO5); no longer JP5.8 (P8)
- net RESET: now also U1.4 (RST)
- net RXD: now also U1.8 (RXD)
- net TXD: now also U1.7 (TXD)
- net CH_PD: no longer names the net of R5.2
- net CH_PD: now also U1.17 (EN); no longer JP4.3 (P3)
- net RESET_5V renamed RESET_3V3
- new net IO0: JP5.6 (P6)
- new net IO12: JP4.6 (P6)
- new net IO13: JP4.7 (P7)
- new net IO14: JP4.5 (P5)
- new net IO15: JP5.4 (P4)
- new net IO16: JP4.4 (P4)
- new net IO2: JP5.5 (P5)
- new net IO4: JP5.7 (P7)
- new net IO5: JP5.8 (P8)
Other:
- moved on the sheet: R5
