File: hardware/glass-break.sch (KiCad schematic (older format))
At the start: 33 parts, among them P1 USB_OTG, SW1 SW_PUSH, SW2 SW_PUSH, SW3 SW_PUSH, U1 ESP-WROOM-02, U11 SPX3819, U2 OP275, U3 electret_microphone

Commit message: update
Connections:
- net GPIO0 is gone; now on net IO0: R2.2, SW1.1, U1.11 (RXD)
- net GPIO12 is gone; now on net IO12: U1.15 (RST)
- net GPIO13 is gone; now on net IO13: U1.14 (IO5)
- net GPIO14 is gone; now on net IO14: U1.16 (TOUT)
- net GPIO15 is gone; now on net IO15: R6.1, U1.13 (GND)
- net GPIO16 is gone; now on net IO16: U1.2 (EN)
- net GPIO2 is gone; now on net IO2: R4.2, U1.12 (TXD)
- net GPIO4 is gone; now on net IO4: SW3.1, U1.9 (GND)
- net +3V3: now also JP5.10 (P10); no longer JP4.3 (P3), JP5.3 (P3)
- net IO0: no longer JP5.6 (P6)
- net IO12: now also JP5.7 (P7); no longer JP4.6 (P6)
- net IO13: now also JP5.6 (P6)
- net IO14: now also JP5.8 (P8); no longer JP4.5 (P5)
- net IO15: no longer JP5.4 (P4)
- net IO16: now also JP4.3 (P3); no longer JP4.4 (P4)
- net IO2: no longer JP5.5 (P5)
- net IO4: no longer JP5.7 (P7)
- net IO5: now also JP4.4 (P4), R8.2, U1.4 (IO13); no longer JP5.8 (P8)
- net RXD_5V: now also JP4.6 (P6); no longer JP5.9 (P9)
- net TXD: now also JP4.5 (P5); no longer JP5.10 (P10)
- net CH_PD: now reaches R5.2, U1.17 (IO16)
- net CH_PD: now also JP5.9 (P9)
- removed net GPIO5: R8.2, U1.4 (IO13)
- new net 1O0: JP5.3 (P3)
- new net I015: JP5.5 (P5)
- new net I02: JP5.4 (P4)
Other:
- moved on the sheet: JP1, JP4, JP5

Commit message: update
Parts:
- removed D1, D2: D, LEDs:LED_0805, symbol D
- removed MBR120-2: ZENER, Diodes_SMD:SOD-123, symbol ZENER
- removed SW1, SW3: SW_PUSH, Buttons_Switches_SMD:SW_SPST_KMR2, symbol SW_PUSH
- added C5, C6, C7, C9: 47pf, Capacitors_SMD:C_0603, symbol C
- added C8: 4.7uF, Capacitors_SMD:C_0805, symbol C
- added D1, D2, D5: LED, LEDs:LED_0805, symbol LED
- added FB1: BLM18PG330SN1D, Resistors_SMD:R_0603, symbol BK0603HS330-T
- added Q1: 2N7002L, TO_SOT_Packages_SMD:SOT-23, symbol Q_NMOS_GSD
- added Q2: BSS84LT1G, TO_SOT_Packages_SMD:SOT-23, symbol Q_PMOS_GSD
- added R13, R20, R21: 1K, Resistors_SMD:R_0603, symbol R
- added R14, R15, R16, R17: 1k, Resistors_SMD:R_0603, symbol R
- added R18, R19: 2.2K, Resistors_SMD:R_0603, symbol R
- added U4: FT230XS, Housings_SSOP:SSOP-16_3.9x4.9mm_Pitch0.635mm, symbol FT230XS
- added U5: TSL2581FN, Housings_DFN_QFN:DFN-6-1EP_2x2mm_Pitch0.65mm, symbol TSL2581FN
- added U6: Si7055-A20-IM, Housings_DFN_QFN:DFN-6-1EP_3x3mm_Pitch0.95mm, symbol Si7055-A20-IM
- C1: value 1uf -> 4.7uf; Part Number (none) -> VJ0805G475KXYTW1BC
- C2: footprint Capacitors_SMD:C_0805 -> Resistors_SMD:R_0603
- C3: footprint Capacitors_SMD:C_0805 -> Capacitors_SMD:C_0603
- D4: Part Number (none) -> LS Q976-NR-1
- MBR120-1: Part Number (none) -> MBR120VLSFT1G
- P1: Part Number (none) -> 10118194-0001LF
- R1, R6: value 10K -> 1K; footprint Resistors_SMD:R_0805 -> Resistors_SMD:R_0603; Part Number (none) -> ERJ-3EKF1001V
- R10, R11, R12, R5, R7, R9: footprint Resistors_SMD:R_0805 -> Resistors_SMD:R_0603
- R2: value 1K -> 27R; footprint Resistors_SMD:R_0805 -> Resistors_SMD:R_0603
- R3: footprint Resistors_SMD:R_0805 -> Resistors_SMD:R_0603; Part Number (none) -> ERJ-3GEYJ103V
- R4: value 10K -> 27R; footprint Resistors_SMD:R_0805 -> Resistors_SMD:R_0603
- R8: footprint Resistors_SMD:R_0805 -> Resistors_SMD:R_0603; Part Number (none) -> ERJ-3EKF1001V
- SW2: Part Number (none) -> KMR211NG LFS
- U11: footprint esp12e:SOT-23-5(MOD) -> TO_SOT_Packages_SMD:SOT-23-5; Part Number (none) -> ERJ-3GEYJ103V
- U3: value electret_microphone -> CMC-5044PF-A
Connections:
- net +BATT is gone; now on net IO4: JP4.9 (P9)
- net 1O0 is gone; now on net IO0: JP5.3 (P3)
- net I015 is gone; now on net IO15: JP5.5 (P5)
- net I02 is gone; now on net IO2: JP5.4 (P4)
- net RXD_5V is gone; now on net RXD: JP1.3 (P3), JP4.6 (P6)
- net +3V3: now also U1.1 (3V3), D1.2 (A), FB1.1, R18.2, R19.2, U5.1 (VDD), U6.5 (VDD); no longer D3.2 (A), R1.1, R4.1, U1.18 (GND)
- net ADC: now also U1.16 (TOUT); no longer U1.3 (IO14)
- net CH_PD: now also U1.2 (EN); no longer U1.17 (IO16)
- net GND: now also R3.2, U1.13 (GND), U1.18 (GND), U1.9 (GND), U11.3 (GND), C5.2, C6.2, C7.2, C8.2, C9.2, Q1.2 (S), U4.13 (GND), U4.5 (GND), U5.2 (ADDR_SEL), U5.3 (GND), U6.2 (GND); no longer R6.2, U1.1 (3V3), U1.10 (IO4), U1.6 (IO15)
- net IO0: now also U1.8 (IO0), R13.1; no longer R2.2, U1.11 (RXD)
- net IO12: now also U1.4 (IO13); no longer U1.15 (RST)
- net IO13: now also U1.4 (IO13); no longer U1.14 (IO5)
- net IO14: now also U1.3 (IO14), R19.1, U5.4 (SCL), U6.6 (SCL); no longer U1.16 (TOUT)
- net IO15: now also U1.6 (IO15); no longer R6.1, U1.13 (GND)
- net IO16: now also JP4.1 (P1), R20.1; no longer JP4.3 (P3), U1.2 (EN)
- net IO2: now also U1.7 (IO2), R18.1, U5.6 (SDA), U6.1 (SDA); no longer R4.2, U1.12 (TXD)
- net IO4: now also R21.1; no longer U1.9 (GND)
- net IO5: now also U1.14 (IO5); no longer U1.4 (IO13)
- net RESET: now also JP4.3 (P3), R1.2, SW2.1, U1.15 (RST), Q2.1 (G), R16.1; no longer U1.4 (IO13)
- net RXD: now also U1.11 (RXD), U4.1 (TXD); no longer U1.8 (IO0)
- net TXD: now also U1.12 (TXD), U4.4 (RXD); no longer U1.7 (IO2)
- net DM: now reaches P1.2 (D-)
- net DM: now also R2.2, C5.1
- net DP: now reaches P1.3 (D+)
- net DP: now also R4.2, C6.1
- net at R2.1: now also U4.9 (USBDM); no longer D3.1 (K)
- removed net RESET_3V3: JP4.1 (P1), R1.2, SW2.1
- new net: D1.1 (K), Q2.2 (S), R1.1
- new net: R21.2, U1.10 (IO4)
- new net: R20.2, U1.17 (IO16)
- new net: FB1.2, U4.12 (VCC)
- new net: C7.1, C9.1, D2.2 (A), D3.2 (A), D5.2 (A), U4.10 (3V3OUT), U4.11 (~RESET), U4.3 (VCCIO)
- new net: R15.2, U4.14 (CBUS1)
- new net: R14.2, U4.15 (CBUS0)
- new net: R17.2, U4.16 (CBUS3)
- new net: R16.2, U4.7 (CBUS2)
- new net: R4.1, U4.8 (USBDP)
- new net: Q2.3 (D), R6.1
- new net: C8.1, Q1.1 (G), R6.2
- new net: Q1.3 (D), R13.2
- new net: D2.1 (K), R14.1
- new net: D3.1 (K), R15.1
- new net: D5.1 (K), R17.1
- new net INT: U5.5 (INT)
Other:
- moved on the sheet: C1, C2, C3, C4, D4, JP1, JP4, JP5, MBR120-1, P1, R1, R10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

Commit message: update
Parts:
- C2: Part Number (none) -> GRM0335C1H120GA01D
- C3: value 10uF -> 10uf; footprint Capacitors_SMD:C_0603 -> Capacitors_SMD:C_0805; Part Number (none) -> VJ0805G106KXQTW1BC
- C4: Part Number (none) -> C0603X5R1C472K030BA
- C5, C6, C7, C9: Part Number (none) -> VJ0603A470JXACW1BC
- D2, D3, D5: Part Number (none) -> LS Q976-NR-1
- FB1: Part Number (none) -> BLM18PG330SN1D
- R10, R12, R5, R9: Part Number (none) -> ERJ-3GEYJ103V
- R11, R18, R19: Part Number (none) -> ERJ-3GEYJ222V
- R14, R15, R16, R17, R20, R21: Part Number (none) -> ERJ-3EKF1001V
- R2, R4: Part Number (none) -> ERJ-3GEYJ270V
- R7: Part Number (none) -> ERJ-3GEYJ105V
- U1: Part Number (none) -> ESP-WROOM-02
- U2: value OP275 -> OPA344; Part Number (none) -> OPA344NA/3K
- U3: Part Number (none) -> CMC-5044PF-A
- U4: Part Number (none) -> FT230XS
- U5: Part Number (none) -> TSL2581FN
- U6: Part Number (none) -> Si7055-A20-IM
Changed lines of the file:
@@
 U 1 1 56C660C8
 P 3550 5150
-F 0 "MBR120-1" H 3550 5250 50  0000 C CNN
+F 0 "MBR120-1" H 3550 5250 50  0001 C CNN
 F 1 "ZENER" H 3550 5050 50  0000 C CNN
 F 2 "Diodes_SMD:SOD-123" H 3550 5150 50  0001 C CNN
@@
 P 10450 3000
 F 0 "C3" H 10475 3100 50  0000 L CNN
-F 1 "10uF" H 10475 2900 50  0000 L CNN
-F 2 "Capacitors_SMD:C_0603" H 10488 2850 50  0001 C CNN
+F 1 "10uf" H 10475 2900 50  0000 L CNN
+F 2 "Capacitors_SMD:C_0805" H 10488 2850 50  0001 C CNN
 F 3 "http://www.mouser.com/ds/2/400/lcc_commercial_general_en-837201.pdf" H 10450 3000 50  0001 C CNN
+F 4 "VJ0805G106KXQTW1BC" H 10450 3000 60  0001 C CNN "Part Number"
 	1    10450 3000
 	-1   0    0    -1
@@
 F 2 "Resistors_SMD:R_0603" H 11438 1400 50  0001 C CNN
 F 3 "GRM0335C1H120GA01D" H 11400 1550 50  0001 C CNN
+F 4 "GRM0335C1H120GA01D" H 11400 1550 60  0001 C CNN "Part Number"
 	1    11400 1550
 	0    1    -1   0
@@
 F 2 "Capacitors_SMD:C_0805" H 10188 2400 50  0001 C CNN
 F 3 "C0603X5R1C472K030BA" H 10150 2550 50  0001 C CNN
+F 4 "C0603X5R1C472K030BA" H 10150 2550 60  0001 C CNN "Part Number"
 	1    10150 2550
 	0    1    -1   0
@@
 F 2 "Resistors_SMD:R_0603" V 11330 1750 50  0001 C CNN
 F 3 "ERJ-3GEYJ105V" H 11400 1750 50  0001 C CNN
+F 4 "ERJ-3GEYJ105V" V 11400 1750 60  0001 C CNN "Part Number"
 	1    11400 1750
 	0    -1   1    0
@@
 F 2 "Resistors_SMD:R_0603" V 10730 3000 50  0001 C CNN
 F 3 "ERJ-3GEYJ103V" H 10800 3000 50  0001 C CNN
+F 4 "ERJ-3GEYJ103V" V 10800 3000 60  0001 C CNN "Part Number"
 	1    10800 3000
 	-1   0    0    -1
@@
 F 2 "Resistors_SMD:R_0603" V 10480 2550 50  0001 C CNN
 F 3 "ERJ-3GEYJ103V" H 10550 2550 50  0001 C CNN
+F 4 "ERJ-3GEYJ103V" V 10550 2550 60  0001 C CNN "Part Number"
 	1    10550 2550
 	0    -1   1    0
@@
 P 11400 2650
 F 0 "U2" H 11400 2800 50  0000 L CNN
-F 1 "OP275" H 11400 2500 50  0000 L CNN
+F 1 "OPA344" H 11400 2500 50  0000 L CNN
 F 2 "Housings_SOIC:SOIC-8_3.9x4.9mm_Pitch1.27mm" H 11300 2700 50  0001 C CNN
 F 3 "http://www.mouser.com/ds/2/609/OP275-879536.pdf" H 11400 2800 50  0001 C CNN
+F 4 "OPA344NA/3K" H 11400 2650 60  0001 C CNN "Part Number"
 	1    11400 2650
 	1    0    0    1
@@
 F 2 "Resistors_SMD:R_0603" V 10730 2300 50  0001 C CNN
 F 3 "ERJ-3GEYJ103V" H 10800 2300 50  0001 C CNN
+F 4 "ERJ-3GEYJ103V" V 10800 2300 60  0001 C CNN "Part Number"
 	1    10800 2300
 	-1   0    0    -1
@@
 F 2 "Resistors_SMD:R_0603" V 9830 2200 50  0001 C CNN
 F 3 "ERJ-3GEYJ222V" H 9900 2200 50  0001 C CNN
+F 4 "ERJ-3GEYJ222V" V 9900 2200 60  0001 C CNN "Part Number"
 	1    9900 2200
 	-1   0    0    -1
@@
 F 2 "esp12e:Electret" H 9000 2900 60  0001 C CNN
 F 3 "http://www.mouser.com/ds/2/670/cmc-5044pf-a-515902.pdf" H 9000 2900 60  0001 C CNN
+F 4 "CMC-5044PF-A" H 9100 2750 60  0001 C CNN "Part Number"
 	1    9100 2750
 	1    0    0    -1
@@
 F 2 "garage-opener:ESP-WROOM-02" H 12450 6800 60  0001 C CNN
 F 3 "http://espressif.com/en/products/hardware/esp-wroom-02/resources" H 12450 6800 60  0001 C CNN
+F 4 "ESP-WROOM-02" H 12450 6800 60  0001 C CNN "Part Number"
 	1    12450 6800
 	1    0    0    -1
@@
 F 2 "Resistors_SMD:R_0603" V 12280 7050 50  0001 C CNN
 F 3 "ERJ-3GEYJ103V" H 12350 7050 50  0001 C CNN
+F 4 "ERJ-3GEYJ103V" V 12350 7050 60  0001 C CNN "Part Number"
 	1    12350 7050
 	1    0    0    -1
@@
 F 2 "Resistors_SMD:R_0603" H 3100 7450 60  0001 C CNN
 F 3 "http://www.murata.com/~/media/webrenewal/support/library/catalog/products/emc/emifil/c31e.ashx?la=en-us" H 3100 7450 60  0001 C CNN
+F 4 "BLM18PG330SN1D" H 3100 7450 60  0001 C CNN "Part Number"
 	1    3100 7450
 	1    0    0    -1
@@
 F 2 "Housings_SSOP:SSOP-16_3.9x4.9mm_Pitch0.635mm" H 3650 8350 50  0001 C CNN
 F 3 "http://www.mouser.com/ds/2/163/DS_FT230X-5395.pdf" H 3650 8350 50  0001 C CNN
+F 4 "FT230XS" H 3650 8350 60  0001 C CNN "Part Number"
 	1    3650 8350
 	1    0    0    -1
@@
 F 2 "Resistors_SMD:R_0603" V 4780 8400 50  0001 C CNN
 F 3 "ERJ-3EKF1001V" H 4850 8400 50  0001 C CNN
+F 4 "ERJ-3EKF1001V" V 4850 8400 60  0001 C CNN "Part Number"
 	1    4850 8400
 	0    1    -1   0
@@
 F 2 "Resistors_SMD:R_0603" V 4780 8550 50  0001 C CNN
 F 3 "ERJ-3EKF1001V" H 4850 8550 50  0001 C CNN
+F 4 "ERJ-3EKF1001V" V 4850 8550 60  0001 C CNN "Part Number"
 	1    4850 8550
 	0    1    -1   0
@@
 F 2 "Resistors_SMD:R_0603" V 4780 8700 50  0001 C CNN
 F 3 "ERJ-3EKF1001V" H 4850 8700 50  0001 C CNN
+F 4 "ERJ-3EKF1001V" V 4850 8700 60  0001 C CNN "Part Number"
 	1    4850 8700
 	0    1    -1   0
@@
 F 2 "Resistors_SMD:R_0603" V 4780 8850 50  0001 C CNN
 F 3 "ERJ-3EKF1001V" H 4850 8850 50  0001 C CNN
+F 4 "ERJ-3EKF1001V" V 4850 8850 60  0001 C CNN "Part Number"
 	1    4850 8850
 	0    1    -1   0
@@
 F 2 "LEDs:LED_0805" H 5450 8400 50  0001 C CNN
 F 3 "LS Q976-NR-1" H 5450 8400 50  0001 C CNN
+F 4 "LS Q976-NR-1" H 5450 8400 60  0001 C CNN "Part Number"
 	1    5450 8400
 	1    0    0    -1
@@
 F 2 "LEDs:LED_0805" H 5450 8550 50  0001 C CNN
 F 3 "LS Q976-NR-1" H 5450 8550 50  0001 C CNN
+F 4 "LS Q976-NR-1" H 5450 8550 60  0001 C CNN "Part Number"
 	1    5450 8550
 	1    0    0    -1
@@
 F 2 "LEDs:LED_0805" H 5450 8850 50  0001 C CNN
 F 3 "LS Q976-NR-1" H 5450 8850 50  0001 C CNN
+F 4 "LS Q976-NR-1" H 5450 8850 60  0001 C CNN "Part Number"
 	1    5450 8850
 	1    0    0    -1
@@
 F 2 "Resistors_SMD:R_0603" V 2630 8150 50  0001 C CNN
 F 3 "ERJ-3GEYJ270V" H 2700 8150 50  0001 C CNN
+F 4 "ERJ-3GEYJ270V" V 2700 8150 60  0001 C CNN "Part Number"
 	1    2700 8150
 	0    1    -1   0
@@
 F 2 "Resistors_SMD:R_0603" V 2630 8350 50  0001 C CNN
 F 3 "ERJ-3GEYJ270V" H 2700 8350 50  0001 C CNN
+F 4 "ERJ-3GEYJ270V" V 2700 8350 60  0001 C CNN "Part Number"
 	1    2700 8350
 	0    1    -1   0
@@
 F 2 "Capacitors_SMD:C_0603" V 2438 8400 50  0001 C CNN
 F 3 "VJ0603A470JXACW1BC" H 2400 8550 50  0001 C CNN
+F 4 "VJ0603A470JXACW1BC" H 2400 8550 60  0001 C CNN "Part Number"
 	1    2400 8550
 	1    0    0    -1
@@
 F 2 "Capacitors_SMD:C_0603" V 2138 8400 50  0001 C CNN
 F 3 "VJ0603A470JXACW1BC" H 2100 8550 50  0001 C CNN
+F 4 "VJ0603A470JXACW1BC" H 2100 8550 60  0001 C CNN "Part Number"
 	1    2100 8550
 	1    0    0    -1
@@
 F 2 "Housings_DFN_QFN:DFN-6-1EP_3x3mm_Pitch0.95mm" H 12050 5050 60  0001 C CNN
 F 3 "http://www.mouser.com/ds/2/368/Si7050-1-3-4-5-A20-907443.pdf" H 12050 5050 60  0001 C CNN
+F 4 "Si7055-A20-IM" H 12500 4750 60  0001 C CNN "Part Number"
 	1    12500 4750
 	1    0    0    -1
@@
 F 2 "Resistors_SMD:R_0603" V 11730 7000 50  0001 C CNN
 F 3 "ERJ-3GEYJ222V" H 11800 7000 50  0001 C CNN
+F 4 "ERJ-3GEYJ222V" V 11800 7000 60  0001 C CNN "Part Number"
 	1    11800 7000
 	1    0    0    1
@@
 F 2 "Resistors_SMD:R_0603" V 11580 7000 50  0001 C CNN
 F 3 "ERJ-3GEYJ222V" H 11650 7000 50  0001 C CNN
+F 4 "ERJ-3GEYJ222V" V 11650 7000 60  0001 C CNN "Part Number"
 	1    11650 7000
 	1    0    0    1
@@
 F 2 "Housings_DFN_QFN:DFN-6-1EP_2x2mm_Pitch0.65mm" H 9050 4550 60  0001 C CNN
 F 3 "http://www.mouser.com/ds/2/588/TSL2581TSL2583-519228.pdf" H 9050 4550 60  0001 C CNN
+F 4 "TSL2581FN" H 9050 4550 60  0001 C CNN "Part Number"
 	1    9050 4550
 	1    0    0    -1
@@
 F 2 "Resistors_SMD:R_0603" V 13930 7250 50  0001 C CNN
 F 3 "ERJ-3EKF1001V" H 14000 7250 50  0001 C CNN
+F 4 "ERJ-3EKF1001V" V 14000 7250 60  0001 C CNN "Part Number"
 	1    14000 7250
 	0    1    1    0
@@
 F 2 "Resistors_SMD:R_0603" V 13930 7950 50  0001 C CNN
 F 3 "ERJ-3EKF1001V" H 14000 7950 50  0001 C CNN
+F 4 "ERJ-3EKF1001V" V 14000 7950 60  0001 C CNN "Part Number"
 	1    14000 7950
 	0    1    1    0
@@
 F 2 "Capacitors_SMD:C_0603" V 2938 9450 50  0001 C CNN
 F 3 "VJ0603A470JXACW1BC" H 2900 9600 50  0001 C CNN
+F 4 "VJ0603A470JXACW1BC" H 2900 9600 60  0001 C CNN "Part Number"
 	1    2900 9600
 	1    0    0    -1
@@
 F 2 "Capacitors_SMD:C_0603" V 2738 9450 50  0001 C CNN
 F 3 "VJ0603A470JXACW1BC" H 2700 9600 50  0001 C CNN
+F 4 "VJ0603A470JXACW1BC" H 2700 9600 60  0001 C CNN "Part Number"
 	1    2700 9600
 	1    0    0    -1
