File: hardware/glass-break.kicad_pcb (KiCad board)
At the start: 2 copper layers, 83.5 x 48.5 mm, 25 parts, among them P1 USB_OTG, U11 SPX3819

Commit message: footprint update
Parts:
- added MBR120-1, MBR120-2: ZENER, Diodes_SMD:SOD-123, F.Cu at (162.8, 103.6)
- added SW1, SW2, SW3: SW_PUSH, Buttons_Switches_SMD:SW_SPST_KMR2, F.Cu at (162.8, 103.6)
- added U1: esp12, esp12e:Esp12e, F.Cu at (147.3, 74.9)
- added U2: OP275, Housings_SOIC:SOIC-8_3.9x4.9mm_Pitch1.27mm, F.Cu at (162.8, 103.6)
- added U3: electret_microphone, esp12e:Electret, F.Cu at (162.8, 103.6)
- C1: value 10UF -> 1uf
- C3: value 1uF -> 10uF
- U11: footprint TO_SOT_Packages_SMD:SC-70-5 -> TO_SOT_Packages_SMD:SOT-23-5
- moved JP5 36.3 mm to (167.6, 55.9), turned to 270 degrees
- moved JP4 23.2 mm to (143.5, 82.5)
Connections:
- JP1 pad 4: GND -> +5V
- JP4 pad 8: GND -> +5V

Commit message: pcd update
Parts:
- moved R7 77.8 mm to (184.5, 62.9), turned to 180 degrees
- moved R11 77.0 mm to (196.6, 62.0), turned to 270 degrees
- moved D2 74.2 mm to (137.2, 61.0), turned to 270 degrees
- moved R3 70.3 mm to (133.1, 71.6), turned to 270 degrees
- moved D3 69.9 mm to (168.8, 62.2), turned to 270 degrees
- moved C4 69.2 mm to (195.6, 69.1), turned to 0 degrees
- moved C2 68.8 mm to (184.5, 59.3)
- moved D4 68.2 mm to (165.2, 67.3), turned to 90 degrees
- moved R8 66.6 mm to (165.2, 72.3), turned to 270 degrees
- moved D1 65.0 mm to (137.2, 76.7), turned to 90 degrees
- moved R2 64.8 mm to (165.5, 62.1), turned to 270 degrees
- moved C1 64.0 mm to (130.0, 71.6), turned to 270 degrees
- moved R10 64.0 mm to (191.4, 69.1), turned to 180 degrees
- moved R12 62.0 mm to (191.0, 62.0), turned to 270 degrees
- moved R6 60.8 mm to (168.4, 67.3), turned to 270 degrees
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Connections:
- D2 pad 1: RXD -> RXD_5V
- JP1 pad 3: RXD -> RXD_5V
- JP5 pad 9: RXD -> RXD_5V
- P1 pad 1: GND -> +5V
- R3 pad 2: LD0_EN -> Net-(R3-Pad2)
- U1 pad 1: RESET_5V -> RESET
- U11 pad 3: LD0_EN -> Net-(R3-Pad2)

Commit message: PCB attempt
Parts:
- moved R5 49.0 mm to (190.6, 119.1)
- moved D4 49.0 mm to (190.6, 109.2), turned to 270 degrees
- moved R1 49.0 mm to (193.8, 119.0)
- moved R4 49.0 mm to (193.8, 114.2)
- moved R6 49.0 mm to (193.8, 109.2)
- moved R8 49.0 mm to (190.6, 114.2)
- moved SW3 49.0 mm to (199.5, 118.2)
- moved D3 49.0 mm to (194.2, 104.1)
- moved R2 49.0 mm to (190.9, 104.0)
- moved SW1 49.0 mm to (199.4, 104.5)
- moved SW2 49.0 mm to (199.4, 111.5)
- moved C3 4.03 mm to (191.8, 70.8)
- moved R7 4.00 mm to (185.7, 59.1)
- moved C2 3.74 mm to (185.7, 62.9)
- moved R9 3.70 mm to (195.6, 71.1)
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Connections:
- P1 pad 6: Net-(P1-Pad6) -> GND
Routing:
- net GND: track 0.00 -> 152.0 mm, vias 0 -> 5
- net +3V3: track 0.00 -> 108.6 mm, vias 0 -> 3
- net ADC: track 0.00 -> 105.8 mm
- net +5V: track 0.00 -> 87.7 mm, vias 0 -> 1
- net RESET_5V: track 0.00 -> 66.3 mm
- net RXD_5V: track 0.00 -> 55.6 mm
- net TXD: track 0.00 -> 49.0 mm
- net +BATT: track 0.00 -> 47.0 mm, vias 0 -> 1
- net GPIO4: track 0.00 -> 32.0 mm
- net GPIO5: track 0.00 -> 27.1 mm
- net RXD: track 0.00 -> 23.9 mm
- net CH_PD: track 0.00 -> 21.8 mm, vias 0 -> 2
- net GPIO2: track 0.00 -> 21.6 mm, vias 0 -> 1
- net GPIO0: track 0.00 -> 21.3 mm, vias 0 -> 1
- net Net-(C3-Pad1): track 0.00 -> 19.2 mm
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- added copper zone on B.Cu, net GND

Commit message: pcb trial2
Parts:
- moved SW2 73.0 mm to (146.1, 61.6), turned to 90 degrees
- moved R1 71.7 mm to (150.0, 62.2)
- moved R5 67.4 mm to (154.2, 62.4)
- moved SW3 66.9 mm to (146.1, 78.1), turned to 90 degrees
- moved SW1 63.6 mm to (146.1, 69.8), turned to 90 degrees
- moved R8 59.6 mm to (154.2, 67.0), turned to 90 degrees
- moved D3 57.6 mm to (150.0, 67.2)
- moved D4 55.2 mm to (150.2, 71.6), turned to 90 degrees
- moved R6 54.0 mm to (150.2, 77.4), turned to 90 degrees
- moved R4 53.9 mm to (154.4, 77.4)
- moved D1 53.6 mm to (185.6, 53.6), turned to 270 degrees
- moved D2 51.8 mm to (185.4, 79.8)
- moved R2 49.1 mm to (154.2, 71.4)
- moved JP4 43.9 mm to (178.4, 55.9), turned to 270 degrees
- moved JP1 37.9 mm to (141.6, 74.9)
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Routing:
- net ADC: track 105.8 -> 32.5 mm
- net GND: track 152.0 -> 110.1 mm, vias 5 -> 0
- net +5V: track 87.7 -> 50.2 mm, vias 1 -> 0
- net +3V3: track 108.6 -> 128.5 mm
- net (no net): track 0.00 -> 19.9 mm
- net GPIO4: track 32.0 -> 12.6 mm
- net RXD_5V: track 55.6 -> 74.8 mm
- net RESET_5V: track 66.3 -> 47.5 mm
- net +BATT: track 47.0 -> 30.3 mm, vias 1 -> 0
- net GPIO0: track 21.3 -> 36.5 mm, vias 1 -> 2
- net Net-(D4-Pad1): track 6.86 -> 16.3 mm
- net TXD: track 49.0 -> 58.0 mm
- net GPIO15: track 14.1 -> 21.3 mm
- net RESET: track 10.3 -> 17.1 mm, vias 0 -> 2
- net Net-(D3-Pad1): track 0.04 -> 6.59 mm
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
Commit message: update
Parts:
- moved R4 3.94 mm to (150.5, 78.0), turned to 90 degrees
- moved R6 3.84 mm to (154.0, 78.0), turned to 270 degrees
Routing:
- net GND: track 110.1 -> 43.7 mm, vias 0 -> 5
- net +3V3: track 128.5 -> 64.3 mm, vias 3 -> 1
- net GPIO15: track 21.3 -> 16.7 mm
- net GPIO2: track 18.5 -> 22.8 mm
- net GPIO0: track 36.5 -> 35.8 mm, vias 2 -> 0
- net RESET_5V: vias 0 -> 1

Commit message: pcb 3
Parts:
- moved D4 5.31 mm to (149.9, 66.3), turned to 180 degrees
- moved D3 4.20 mm to (149.9, 71.3), turned to 180 degrees
- moved R12 3.35 mm to (191.6, 65.5)
- moved C4 3.18 mm to (195.4, 69.8)
- moved R4 3.08 mm to (149.8, 75.0), turned to 0 degrees
- moved R10 3.08 mm to (191.6, 69.8)
- moved C3 3.05 mm to (191.8, 73.9)
- moved R6 3.00 mm to (154.0, 75.0), turned to 180 degrees
- moved R9 2.88 mm to (195.5, 74.0)
- moved R11 2.83 mm to (195.5, 65.3)
- moved R1 0.69 mm to (150.6, 62.6), turned to 0 degrees
- moved R8 0.60 mm to (154.2, 66.4), turned to 0 degrees
- moved R2 0.29 mm to (153.9, 71.2), turned to 0 degrees
- turned R5 to 0 degrees
Routing:
- net +3V3: track 64.3 -> 100.3 mm, vias 1 -> 2
- net GPIO4: track 12.6 -> 41.7 mm
- net Net-(D4-Pad1): track 16.3 -> 2.29 mm
- net RESET_5V: track 47.5 -> 56.7 mm
- net GND: track 43.7 -> 36.7 mm, vias 5 -> 7
- net Net-(D3-Pad1): track 6.59 -> 2.14 mm
- net Net-(C3-Pad1): track 20.1 -> 15.7 mm
- net GPIO15: track 16.7 -> 14.6 mm
- net Net-(C2-Pad2): track 12.3 -> 14.2 mm
- net Net-(C4-Pad2): track 8.56 -> 10.2 mm
- net GPIO0: track 35.8 -> 37.1 mm, vias 0 -> 2
- net GPIO5: track 27.8 -> 26.7 mm
- net GPIO2: track 22.8 -> 21.8 mm
- net RESET: track 17.1 -> 17.6 mm

Commit message: pcb 3
Parts:
- moved JP1 0.11 mm to (141.5, 74.9)
Routing:
- net +5V: track 50.2 -> 49.2 mm
Changed lines of the file:
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@@
     (links 84)
     (no_connects 6)
-    (area 119.551 44.399999 221 207.500161)
+    (area 120.924999 44.924999 204.575001 93.575001)
     (thickness 1.6)
     (drawings 35)
@@
     (add_net TXD)
   )
+  (module Pin_Headers:Pin_Header_Straight_1x06 (layer F.Cu)
+    (at 141.5 74.9 180)
+    (descr "Through hole pin header")
+    (tags "pin header")
+    (fp_text reference JP1 (at 0 -5.1 180) (layer F.SilkS)
+      (effects (font (size 1 1) (thickness 0.15)))
+    )
+    (fp_text value CONN_01X06 (at 0 -3.1 180) (layer F.Fab)
+      (effects (font (size 1 1) (thickness 0.15)))
+    )
+    (fp_line (start -1.75 -1.75) (end -1.75 14.45) (layer F.CrtYd) (width 0.05))
+    (fp_line (start 1.75 -1.75) (end 1.75 14.45) (layer F.CrtYd) (width 0.05))
+    (fp_line (start -1.75 -1.75) (end 1.75 -1.75) (layer F.CrtYd) (width 0.05))
+    (fp_line (start -1.75 14.45) (end 1.75 14.45) (layer F.CrtYd) (width 0.05))
+    (fp_line (start 1.27 1.27) (end 1.27 13.97) (layer F.SilkS) (width 0.15))
+    (fp_line (start 1.27 13.97) (end -1.27 13.97) (layer F.SilkS) (width 0.15))
+    (fp_line (start -1.27 13.97) (end -1.27 1.27) (layer F.SilkS) (width 0.15))
+    (fp_line (start 1.55 -1.55) (end 1.55 0) (layer F.SilkS) (width 0.15))
+    (fp_line (start 1.27 1.27) (end -1.27 1.27) (layer F.SilkS) (width 0.15))
+    (fp_line (start -1.55 0) (end -1.55 -1.55) (layer F.SilkS) (width 0.15))
+    (fp_line (start -1.55 -1.55) (end 1.55 -1.55) (layer F.SilkS) (width 0.15))
+    (pad 1 thru_hole rect (at 0 0 180) (size 2.032 1.7272) (drill 1.016) (layers *.Cu *.Mask F.SilkS)
+      (net 12 "Net-(JP1-Pad1)"))
+    (pad 2 thru_hole oval (at 0 2.54 180) (size 2.032 1.7272) (drill 1.016) (layers *.Cu *.Mask F.SilkS)
+      (net 13 TXD))
+    (pad 3 thru_hole oval (at 0 5.08 180) (size 2.032 1.7272) (drill 1.016) (layers *.Cu *.Mask F.SilkS)
+      (net 21 RXD_5V))
+    (pad 4 thru_hole oval (at 0 7.62 180) (size 2.032 1.7272) (drill 1.016) (layers *.Cu *.Mask F.SilkS)
+      (net 17 +5V))
+    (pad 5 thru_hole oval (at 0 10.16 180) (size 2.032 1.7272) (drill 1.016) (layers *.Cu *.Mask F.SilkS)
+      (net 14 "Net-(JP1-Pad5)"))
+    (pad 6 thru_hole oval (at 0 12.7 180) (size 2.032 1.7272) (drill 1.016) (layers *.Cu *.Mask F.SilkS)
+      (net 2 GND))
+    (model Pin_Headers.3dshapes/Pin_Header_Straight_1x06.wrl
+      (at (xyz 0 -0.25 0))
+      (scale (xyz 1 1 1))
+      (rotate (xyz 0 0 90))
+    )
+  )
   (module Resistors_SMD:R_0805 (layer F.Cu)
     (at 153.95 71.25)
@@
     (model Pin_Headers.3dshapes/Pin_Header_Straight_1x10.wrl
       (at (xyz 0 -0.45 0))
-      (scale (xyz 1 1 1))
-      (rotate (xyz 0 0 90))
-    )
-  )
-  (module Pin_Headers:Pin_Header_Straight_1x06 (layer F.Cu)
-    (at 141.605 74.93 180)
-    (descr "Through hole pin header")
-    (tags "pin header")
-    (fp_text reference JP1 (at 0 -5.1 180) (layer F.SilkS)
-      (effects (font (size 1 1) (thickness 0.15)))
-    )
-    (fp_text value CONN_01X06 (at 0 -3.1 180) (layer F.Fab)
-      (effects (font (size 1 1) (thickness 0.15)))
-    )
-    (fp_line (start -1.75 -1.75) (end -1.75 14.45) (layer F.CrtYd) (width 0.05))
-    (fp_line (start 1.75 -1.75) (end 1.75 14.45) (layer F.CrtYd) (width 0.05))
-    (fp_line (start -1.75 -1.75) (end 1.75 -1.75) (layer F.CrtYd) (width 0.05))
-    (fp_line (start -1.75 14.45) (end 1.75 14.45) (layer F.CrtYd) (width 0.05))
-    (fp_line (start 1.27 1.27) (end 1.27 13.97) (layer F.SilkS) (width 0.15))
-    (fp_line (start 1.27 13.97) (end -1.27 13.97) (layer F.SilkS) (width 0.15))
-    (fp_line (start -1.27 13.97) (end -1.27 1.27) (layer F.SilkS) (width 0.15))
-    (fp_line (start 1.55 -1.55) (end 1.55 0) (layer F.SilkS) (width 0.15))
-    (fp_line (start 1.27 1.27) (end -1.27 1.27) (layer F.SilkS) (width 0.15))
-    (fp_line (start -1.55 0) (end -1.55 -1.55) (layer F.SilkS) (width 0.15))
-    (fp_line (start -1.55 -1.55) (end 1.55 -1.55) (layer F.SilkS) (width 0.15))
-    (pad 1 thru_hole rect (at 0 0 180) (size 2.032 1.7272) (drill 1.016) (layers *.Cu *.Mask F.SilkS)
-      (net 12 "Net-(JP1-Pad1)"))
-    (pad 2 thru_hole oval (at 0 2.54 180) (size 2.032 1.7272) (drill 1.016) (layers *.Cu *.Mask F.SilkS)
-      (net 13 TXD))
-    (pad 3 thru_hole oval (at 0 5.08 180) (size 2.032 1.7272) (drill 1.016) (layers *.Cu *.Mask F.SilkS)
-      (net 21 RXD_5V))
-    (pad 4 thru_hole oval (at 0 7.62 180) (size 2.032 1.7272) (drill 1.016) (layers *.Cu *.Mask F.SilkS)
-      (net 17 +5V))
-    (pad 5 thru_hole oval (at 0 10.16 180) (size 2.032 1.7272) (drill 1.016) (layers *.Cu *.Mask F.SilkS)
-      (net 14 "Net-(JP1-Pad5)"))
-    (pad 6 thru_hole oval (at 0 12.7 180) (size 2.032 1.7272) (drill 1.016) (layers *.Cu *.Mask F.SilkS)
-      (net 2 GND))
-    (model Pin_Headers.3dshapes/Pin_Header_Straight_1x06.wrl
-      (at (xyz 0 -0.25 0))
       (scale (xyz 1 1 1))
       (rotate (xyz 0 0 90))
@@
   (segment (start 136.06 71.94) (end 135.5 72.5) (width 0.25) (layer F.Cu) (net 2))
   (via (at 135.5 72.5) (size 0.6) (drill 0.4) (layers F.Cu B.Cu) (net 2))
-  (segment (start 141.605 62.23) (end 141.7574 62.23) (width 0.25) (layer F.Cu) (net 2))
   (segment (start 146.85 63.695) (end 146.85 63.645) (width 0.25) (layer F.Cu) (net 2))
   (segment (start 146.85 59.545) (end 146.85 59.495) (width 0.25) (layer F.Cu) (net 2))
@@
   (segment (start 158.115 55.7276) (end 158.115 55.88) (width 0.25) (layer F.Cu) (net 15))
   (segment (start 133.239 64.135) (end 133.096 64.278) (width 0.25) (layer F.Cu) (net 15))
+  (segment (start 147.462662 54.53899) (end 144.474999 57.526653) (width 0.25) (layer F.Cu) (net 17))
+  (segment (start 144.474999 57.526653) (end 144.474999 64.457401) (width 0.25) (layer F.Cu) (net 17))
+  (segment (start 144.474999 64.457401) (end 141.6524 67.28) (width 0.25) (layer F.Cu) (net 17))
+  (segment (start 141.6524 67.28) (end 141.5 67.28) (width 0.25) (layer F.Cu) (net 17))
   (segment (start 141.605 67.31) (end 141.4526 67.31) (width 0.25) (layer F.Cu) (net 17))
   (segment (start 147.462662 54.53899) (end 156.067338 54.53899) (width 0.25) (layer F.Cu) (net 17))
-  (segment (start 141.4526 67.31) (end 140.26399 66.12139) (width 0.25) (layer F.Cu) (net 17))
-  (segment (start 140.26399 66.12139) (end 140.26399 61.737662) (width 0.25) (layer F.Cu) (net 17))
-  (segment (start 140.26399 61.737662) (end 147.462662 54.53899) (width 0.25) (layer F.Cu) (net 17))
   (segment (start 156.92639 56.524738) (end 157.622662 57.22101) (width 0.25) (layer F.Cu) (net 17))
   (segment (start 156.067338 54.53899) (end 156.92639 55.398042) (width 0.25) (layer F.Cu) (net 17))

Commit message: update
Parts:
- moved MBR120-1 3.72 mm to (130.0, 69.8)
- moved C1 3.17 mm to (129.9, 74.8), turned to 90 degrees
- moved R3 3.02 mm to (133.2, 74.7), turned to 90 degrees
- moved MBR120-2 2.32 mm to (133.2, 68.2)
- moved SW2 1.40 mm to (146.1, 63.0), turned to 270 degrees
- moved U11 1.00 mm to (137.2, 70.6)
- moved D2 0.95 mm to (185.4, 78.8), turned to 90 degrees
Routing:
- net RXD_5V: track 74.8 -> 58.1 mm, vias 0 -> 1
- net +5V: track 49.2 -> 39.8 mm
- net RESET_5V: track 56.7 -> 47.9 mm
- net Net-(C1-Pad1): track 12.9 -> 15.2 mm
- net RXD: track 17.5 -> 16.7 mm
- net +BATT: track 30.3 -> 29.6 mm
