File: hardware/glass-break.kicad_pcb (KiCad board)
At the start: 2 copper layers, 83.5 x 48.5 mm, 33 parts, among them P1 USB_OTG, SW1 SW_PUSH, SW2 SW_PUSH, SW3 SW_PUSH, U1 esp12, U11 SPX3819, U2 OP275, U3 electret_microphone

Commit message: update
Parts:
- moved C1 11.0 mm to (131.2, 63.9)
- moved R11 6.16 mm to (201.2, 62.9)
- moved MBR120-2 5.58 mm to (136.2, 63.5)
- moved C4 5.01 mm to (196.2, 64.9), turned to 90 degrees
- moved R9 3.26 mm to (198.2, 75.9)
- moved R12 2.61 mm to (192.2, 63.0)
- moved C3 2.25 mm to (192.4, 76.0)
- moved MBR120-1 1.32 mm to (131.2, 69.0)
- moved R10 1.25 mm to (192.1, 70.9)
- moved R3 1.25 mm to (134.2, 73.9), turned to 0 degrees
- moved R1 0.70 mm to (150.6, 61.9), turned to 90 degrees
- moved U11 0.70 mm to (137.2, 69.9)
- moved R5 0.50 mm to (154.2, 61.9), turned to 90 degrees
Routing:
- net CH_PD: track 23.2 -> 8.73 mm
- net GND: track 36.3 -> 27.0 mm, vias 7 -> 9
- net Net-(C3-Pad1): track 15.7 -> 20.4 mm
- net +BATT: track 29.6 -> 25.1 mm
- net Net-(C4-Pad1): track 1.89 -> 6.36 mm
- net Net-(C1-Pad1): track 15.2 -> 19.6 mm, vias 0 -> 2
- net +3V3: track 100.7 -> 98.0 mm
- net RESET_5V: track 47.9 -> 46.5 mm
- net Net-(C2-Pad2): track 14.2 -> 15.4 mm
- net Net-(C4-Pad2): track 10.2 -> 9.22 mm

Commit message: update
Routing:
- net (no net): track 19.9 -> 0.00 mm
Changed lines of the file:
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@@
 (kicad_pcb (version 4) (host pcbnew 4.0.2-4+6225~38~ubuntu15.10.1-stable)
   (general
-    (links 84)
-    (no_connects 3)
-    (area 120.924999 44.924999 204.575001 93.575001)
+    (links 95)
+    (no_connects 14)
+    (area 119.551 44.399999 221 119.508333)
     (thickness 1.6)
     (drawings 35)
-    (tracks 300)
+    (tracks 298)
     (zones 0)
     (modules 33)
@@
     (47 F.CrtYd user)
     (48 B.Fab user)
-    (49 F.Fab user)
+    (49 F.Fab user hide)
   )
   (setup
@@
     (add_net "Net-(D3-Pad1)")
     (add_net "Net-(D4-Pad1)")
+    (add_net "Net-(D5-Pad1)")
+    (add_net "Net-(D5-Pad2)")
     (add_net "Net-(JP1-Pad1)")
     (add_net "Net-(JP1-Pad5)")
@@
     (add_net "Net-(P1-Pad3)")
     (add_net "Net-(P1-Pad4)")
+    (add_net "Net-(P2-Pad4)")
+    (add_net "Net-(P2-Pad5)")
+    (add_net "Net-(Q1-Pad1)")
     (add_net "Net-(R3-Pad2)")
     (add_net "Net-(U11-Pad4)")
@@
   (gr_line (start 205 94.5) (end 205 44.5) (angle 90) (layer Margin) (width 0.2))
   (gr_line (start 120.5 94.5) (end 205 94.5) (angle 90) (layer Margin) (width 0.2))
-  (segment (start 128.237027 207.175159) (end 126.260375 205.198507) (width 0.25) (layer B.Cu) (net 0))
-  (segment (start 145.310375 207.175159) (end 128.237027 207.175159) (width 0.25) (layer B.Cu) (net 0))
   (segment (start 133.2 71.02) (end 133.65 70.57) (width 0.25) (layer F.Cu) (net 1))
   (segment (start 133.65 70.57) (end 135.27 68.95) (width 0.25) (layer F.Cu) (net 1))

Commit message: update
Routing:
- net CH_PD: track 8.73 -> 25.7 mm, vias 0 -> 2
Changed lines of the file:
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@@
 (kicad_pcb (version 4) (host pcbnew 4.0.2-4+6225~38~ubuntu15.10.1-stable)
   (general
-    (links 95)
-    (no_connects 14)
-    (area 119.551 44.399999 221 119.508333)
+    (links 84)
+    (no_connects 2)
+    (area 119.551 44.399999 221 102.200001)
     (thickness 1.6)
     (drawings 35)
-    (tracks 298)
+    (tracks 306)
     (zones 0)
     (modules 33)
@@
     (add_net "Net-(D3-Pad1)")
     (add_net "Net-(D4-Pad1)")
-    (add_net "Net-(D5-Pad1)")
-    (add_net "Net-(D5-Pad2)")
     (add_net "Net-(JP1-Pad1)")
     (add_net "Net-(JP1-Pad5)")
@@
     (add_net "Net-(P1-Pad3)")
     (add_net "Net-(P1-Pad4)")
-    (add_net "Net-(P2-Pad4)")
-    (add_net "Net-(P2-Pad5)")
-    (add_net "Net-(Q1-Pad1)")
     (add_net "Net-(R3-Pad2)")
     (add_net "Net-(U11-Pad4)")
@@
   (segment (start 150.99804 66.3) (end 153.15 66.3) (width 0.25) (layer F.Cu) (net 24))
   (segment (start 153.15 66.3) (end 153.25 66.4) (width 0.25) (layer F.Cu) (net 24))
+  (segment (start 154.15 60.95) (end 156.05 60.95) (width 0.25) (layer F.Cu) (net 25) (status 400000))
+  (segment (start 167.75 63.95) (end 168.72 62.98) (width 0.25) (layer F.Cu) (net 25) (status 800000))
+  (via (at 167.75 63.95) (size 0.6) (drill 0.4) (layers F.Cu B.Cu) (net 25))
+  (segment (start 159.05 63.95) (end 167.75 63.95) (width 0.25) (layer B.Cu) (net 25))
+  (segment (start 156.8 61.7) (end 159.05 63.95) (width 0.25) (layer B.Cu) (net 25))
+  (via (at 156.8 61.7) (size 0.6) (drill 0.4) (layers F.Cu B.Cu) (net 25))
+  (segment (start 156.05 60.95) (end 156.8 61.7) (width 0.25) (layer F.Cu) (net 25))
+  (segment (start 168.72 62.98) (end 168.72 62.23) (width 0.25) (layer F.Cu) (net 25) (status C00000))
   (segment (start 168.72 62.605) (end 168.72 62.23) (width 0.25) (layer F.Cu) (net 25))
   (segment (start 168.72 62.23) (end 168.72 60.515) (width 0.25) (layer F.Cu) (net 25))

Commit message: update
Parts:
- U1: value esp12 -> ESP-WROOM-02; footprint esp12e:Esp12e -> garage-opener:ESP-WROOM-02
- moved U1 63.7 mm to (166.2, 125.6), turned to 0 degrees
- moved D2 4.22 mm to (185.1, 83.0)
- moved R9 2.17 mm to (196.1, 76.5)
- moved U3 2.09 mm to (201.0, 70.7)
- moved C4 2.07 mm to (196.4, 62.9)
- moved R10 1.86 mm to (193.2, 69.4)
- moved C3 0.92 mm to (191.6, 76.4)
Connections:
- R5 pad 2: CH_PD -> Net-(R5-Pad2)
- U1 pad 1: RESET -> GND
- U1 pad 10: GPIO15 -> GND
- U1 pad 11: GPIO2 -> GPIO0
- U1 pad 12: GPIO0 -> GPIO2
- U1 pad 13: GPIO4 -> GPIO15
- U1 pad 14: GPIO5 -> GPIO13
- U1 pad 15: RXD -> GPIO12
- U1 pad 16: TXD -> GPIO14
- U1 pad 2: ADC -> GPIO16
- U1 pad 3: CH_PD -> ADC
- U1 pad 4: GPIO16 -> RESET
- U1 pad 5: GPIO14 -> GPIO5
- U1 pad 6: GPIO12 -> GND
- U1 pad 7: GPIO13 -> TXD
- U1 pad 8: +3V3 -> RXD
- U1 pad 9: GND -> GPIO4
Routing:
- net +3V3: track 98.0 -> 0.00 mm, vias 2 -> 0
- net RXD_5V: track 58.1 -> 0.00 mm, vias 1 -> 0
- net TXD: track 58.0 -> 0.00 mm
- net RESET_5V: track 46.5 -> 0.00 mm, vias 1 -> 0
- net GPIO4: track 41.7 -> 0.00 mm
- net +5V: track 39.8 -> 0.00 mm
- net GPIO0: track 37.1 -> 0.00 mm, vias 2 -> 0
- net ADC: track 32.5 -> 0.00 mm
- net GND: track 27.0 -> 0.00 mm, vias 9 -> 0
- net GPIO5: track 26.7 -> 0.00 mm
- net CH_PD: track 25.7 -> 0.00 mm, vias 2 -> 0
- net +BATT: track 25.1 -> 0.00 mm
- net GPIO2: track 21.8 -> 0.00 mm
- net Net-(C3-Pad1): track 20.4 -> 0.00 mm
- net Net-(C1-Pad1): track 19.6 -> 0.00 mm, vias 2 -> 0
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
Commit message: update
Parts:
- moved U1 66.5 mm to (174.2, 59.6), turned to 270 degrees
- moved D2 34.6 mm to (157.7, 61.9), turned to 270 degrees
- moved R11 9.96 mm to (194.7, 70.5)
- moved D3 7.56 mm to (150.2, 78.9)
- moved R12 7.47 mm to (191.2, 70.3)
- moved R2 7.34 mm to (155.6, 78.4)
- moved R5 6.63 mm to (153.2, 68.5), turned to 270 degrees
- moved U11 6.58 mm to (133.7, 75.5), turned to 270 degrees
- moved R10 4.49 mm to (191.2, 65.4), turned to 90 degrees
- moved R8 4.47 mm to (154.7, 62.0), turned to 90 degrees
- moved R3 4.27 mm to (135.7, 69.9), turned to 270 degrees
- moved R4 3.40 mm to (153.2, 74.9)
- moved D4 3.18 mm to (153.1, 65.9)
- moved R6 3.15 mm to (153.2, 71.9)
- moved C4 3.14 mm to (195.7, 65.9), turned to 0 degrees
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Connections:
- net RESET_5V renamed RESET_3V3
- JP4 pad 3: CH_PD -> IO16
- JP4 pad 4: GPIO16 -> IO5
- JP4 pad 5: GPIO14 -> TXD
- JP4 pad 6: GPIO12 -> RXD_5V
- JP4 pad 7: GPIO13 -> IO13
- JP5 pad 10: TXD -> +3V3
- JP5 pad 2: LD0_EN -> GND
- JP5 pad 3: +3V3 -> 1O0
- JP5 pad 4: GPIO15 -> I02
- JP5 pad 5: GPIO2 -> I015
- JP5 pad 6: GPIO0 -> IO13
- JP5 pad 7: GPIO4 -> IO12
- JP5 pad 8: GPIO5 -> IO14
- JP5 pad 9: RXD_5V -> CH_PD
- R2 pad 2: GPIO0 -> IO0
- R4 pad 2: GPIO2 -> IO2
- R5 pad 2: Net-(R5-Pad2) -> CH_PD
- R6 pad 1: GPIO15 -> IO15
- R8 pad 2: GPIO5 -> IO5
- SW1 pad 1: GPIO0 -> IO0
- SW3 pad 1: GPIO4 -> IO4
- U1 pad 11: GPIO0 -> IO0
- U1 pad 12: GPIO2 -> IO2
- U1 pad 13: GPIO15 -> IO15
- U1 pad 14: GPIO13 -> IO13
- U1 pad 15: GPIO12 -> IO12
- U1 pad 16: GPIO14 -> IO14
- U1 pad 17: Net-(R5-Pad2) -> CH_PD
- U1 pad 2: GPIO16 -> IO16
- U1 pad 5: GPIO5 -> IO5
- U1 pad 9: GPIO4 -> IO4
Routing:
- net +3V3: track 0.00 -> 98.2 mm
- net RESET_3V3: track 0.00 -> 49.9 mm, vias 0 -> 1
- net +5V: track 0.00 -> 44.9 mm, vias 0 -> 1
- net GND: track 0.00 -> 40.2 mm, vias 0 -> 10
- net TXD: track 0.00 -> 34.3 mm, vias 0 -> 1
- net IO4: track 0.00 -> 32.2 mm
- net RXD_5V: track 0.00 -> 30.7 mm, vias 0 -> 1
- net CH_PD: track 0.00 -> 30.6 mm
- net IO13: track 0.00 -> 29.9 mm, vias 0 -> 1
- net ADC: track 0.00 -> 27.1 mm
- net IO0: track 0.00 -> 26.4 mm, vias 0 -> 2
- net +BATT: track 0.00 -> 26.4 mm
- net IO5: track 0.00 -> 23.4 mm, vias 0 -> 2
- net RESET: track 0.00 -> 20.9 mm
- net Net-(C1-Pad1): track 0.00 -> 19.0 mm
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
Commit message: update
Parts:
- removed MBR120-2: ZENER, Diodes_SMD:SOD-123
- removed SW1, SW3: SW_PUSH, Buttons_Switches_SMD:SW_SPST_KMR2
- added C5: 47pf, Capacitors_SMD:C_0603, F.Cu at (135.0, 71.7)
- added C6: 47pf, Capacitors_SMD:C_0603, F.Cu at (136.7, 60.2)
- added C7: 47pf, Capacitors_SMD:C_0603, F.Cu at (142.9, 59.9)
- added C8: 4.7uF, Capacitors_SMD:C_0805, F.Cu at (146.7, 78.2)
- added C9: 47pf, Capacitors_SMD:C_0603, F.Cu at (145.1, 59.9)
- added D5: LED, LEDs:LED_0805, F.Cu at (141.2, 76.3)
- added FB1: BLM18PG330SN1D, Resistors_SMD:R_0603, F.Cu at (136.7, 65.3)
- added Q1: 2N7002L, TO_SOT_Packages_SMD:SOT-23, F.Cu at (148.3, 83.3)
- added Q2: BSS84LT1G, TO_SOT_Packages_SMD:SOT-23, F.Cu at (148.4, 73.4)
- added R13: 1K, Resistors_SMD:R_0603, F.Cu at (187.4, 63.0)
- added R14: 1k, Resistors_SMD:R_0603, F.Cu at (141.0, 71.7)
- added R15: 1k, Resistors_SMD:R_0603, F.Cu at (139.1, 71.8)
- added R16: 1k, Resistors_SMD:R_0603, F.Cu at (141.0, 60.0)
- added R17: 1k, Resistors_SMD:R_0603, F.Cu at (142.9, 71.7)
- added R18: 2.2K, Resistors_SMD:R_0603, F.Cu at (187.4, 65.5)
- added R19: 2.2K, Resistors_SMD:R_0603, F.Cu at (187.3, 79.6)
- added R20: 1K, Resistors_SMD:R_0603, F.Cu at (156.6, 68.5)
- added R21: 1K, Resistors_SMD:R_0603, F.Cu at (157.0, 57.1)
- added U4: FT230XS, Housings_SSOP:SSOP-16_3.9x4.9mm_Pitch0.635mm, F.Cu at (141.0, 65.6)
- added U5: TSL2581FN, Housings_DFN_QFN:DFN-6-1EP_2x2mm_Pitch0.65mm, F.Cu at (188.9, 75.2)
- added U6: Si7055-A20-IM, Housings_DFN_QFN:DFN-6-1EP_3x3mm_Pitch0.95mm, F.Cu at (193.5, 75.4)
- C1: value 1uf -> 4.7uf
- C2: footprint Capacitors_SMD:C_0805 -> Resistors_SMD:R_0603
- C3, C4: footprint Capacitors_SMD:C_0805 -> Capacitors_SMD:C_0603
- D1, D2: value D -> LED
- R1, R6: value 10K -> 1K; footprint Resistors_SMD:R_0805 -> Resistors_SMD:R_0603
- R10, R11, R12, R3, R5, R7, R8, R9: footprint Resistors_SMD:R_0805 -> Resistors_SMD:R_0603
- R2: value 1K -> 27R; footprint Resistors_SMD:R_0805 -> Resistors_SMD:R_0603
- R4: value 10K -> 27R; footprint Resistors_SMD:R_0805 -> Resistors_SMD:R_0603
- U3: value electret_microphone -> CMC-5044PF-A
- moved R5 40.3 mm to (193.3, 71.9), turned to 180 degrees
- moved D1 39.5 mm to (148.3, 66.5), turned to 0 degrees
- moved R9 37.5 mm to (158.1, 85.0), turned to 0 degrees
- moved JP5 37.1 mm to (183.1, 58.0), turned to 0 degrees
- moved JP1 36.7 mm to (168.7, 50.2), turned to 270 degrees
- moved C4 36.1 mm to (166.1, 86.7), turned to 270 degrees
- moved R11 35.2 mm to (163.6, 86.9)
- moved R12 35.1 mm to (158.0, 82.0), turned to 180 degrees
- moved JP4 35.1 mm to (153.6, 80.6), turned to 180 degrees
- moved C3 35.0 mm to (158.2, 88.1), turned to 0 degrees
- moved R7 33.1 mm to (159.2, 78.8), turned to 90 degrees
- moved C2 32.9 mm to (156.9, 78.8), turned to 270 degrees
- moved R10 31.1 mm to (168.4, 86.7)
- moved D2 24.3 mm to (138.1, 76.3)
- moved U3 24.0 mm to (183.7, 86.5), turned to 0 degrees
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Connections:
- D1 pad 1: RESET_3V3 -> Net-(D1-Pad1)
- D1 pad 2: RESET -> +3V3
- D2 pad 1: RXD_5V -> Net-(D2-Pad1)
- D2 pad 2: RXD -> Net-(C7-Pad1)
- D3 pad 2: +3V3 -> Net-(C7-Pad1)
- JP1 pad 3: RXD_5V -> RXD
- JP4 pad 1: RESET_3V3 -> IO16
- JP4 pad 3: IO16 -> RESET
- JP4 pad 6: RXD_5V -> RXD
- JP4 pad 9: +BATT -> IO4
- JP5 pad 3: 1O0 -> IO0
- JP5 pad 4: I02 -> IO2
- JP5 pad 5: I015 -> IO15
- P1 pad 2: Net-(P1-Pad2) -> DM
- P1 pad 3: Net-(P1-Pad3) -> DP
- R1 pad 1: +3V3 -> Net-(D1-Pad1)
- R1 pad 2: RESET_3V3 -> RESET
- R2 pad 1: Net-(D3-Pad1) -> Net-(R2-Pad1)
- R2 pad 2: IO0 -> DM
- R3 pad 2: Net-(R3-Pad2) -> GND
- R4 pad 1: +3V3 -> Net-(R4-Pad1)
- R4 pad 2: IO2 -> DP
- R6 pad 1: IO15 -> Net-(Q2-Pad3)
- R6 pad 2: GND -> Net-(C8-Pad1)
- SW2 pad 1: RESET_3V3 -> RESET
- U1 pad 1: GND -> +3V3
- U1 pad 10: GND -> Net-(R21-Pad2)
- U1 pad 11: IO0 -> RXD
- U1 pad 12: IO2 -> TXD
- U1 pad 13: IO15 -> GND
- U1 pad 14: IO13 -> IO5
- U1 pad 15: IO12 -> RESET
- U1 pad 16: IO14 -> ADC
- U1 pad 17: CH_PD -> Net-(R20-Pad2)
- U1 pad 18: +3V3 -> GND
- U1 pad 2: IO16 -> CH_PD
- U1 pad 3: ADC -> IO14
- U1 pad 4: RESET -> IO12
- U1 pad 5: IO5 -> (no net)
- U1 pad 6: GND -> IO15
- U1 pad 7: TXD -> IO2
- U1 pad 8: RXD -> IO0
- U1 pad 9: IO4 -> GND
- U11 pad 3: Net-(R3-Pad2) -> GND
Routing:
- net Net-(Q1-Pad3): track 0.00 -> 50.6 mm, vias 0 -> 2
- net RESET_3V3: track 49.9 -> 0.00 mm, vias 1 -> 0
- net +3V3: track 98.2 -> 147.8 mm, vias 0 -> 11
- net RXD: track 6.72 -> 43.7 mm
- net RESET: track 20.9 -> 53.3 mm, vias 0 -> 3
- net RXD_5V: track 30.7 -> 0.00 mm, vias 1 -> 0
- net IO4: track 32.2 -> 4.71 mm
- net Net-(C7-Pad1): track 0.00 -> 27.3 mm, vias 0 -> 4
- net +BATT: track 26.4 -> 0.00 mm
- net DP: track 0.00 -> 23.1 mm
- net IO14: track 6.85 -> 28.4 mm, vias 0 -> 2
- net IO0: track 26.4 -> 11.5 mm, vias 2 -> 0
- net IO2: track 12.5 -> 26.4 mm, vias 0 -> 2
- net DM: track 0.00 -> 12.3 mm
- net Net-(C1-Pad1): track 19.0 -> 9.37 mm
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Other:
- board text added: "pyfi, llc andy@pyfi.org"

Commit message: update
Parts:
- C3: value 10uF -> 10uf; footprint Capacitors_SMD:C_0603 -> Capacitors_SMD:C_0805
- moved C3 0.12 mm to (158.2, 88.2)
Routing:
- net GND: track 35.3 -> 35.2 mm, vias 20 -> 21
Changed lines of the file:
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@@
   (general
     (links 125)
-    (no_connects 1)
+    (no_connects 3)
     (area 120.924999 44.924999 204.575001 93.575001)
     (thickness 1.6)
     (drawings 36)
-    (tracks 496)
+    (tracks 499)
     (zones 0)
     (modules 51)
@@
   )
   (module Capacitors_SMD:C_0603 (layer F.Cu)
-    (at 158.18 88.08)
-    (descr "Capacitor SMD 0603, reflow soldering, AVX (see smccp.pdf)")
-    (tags "capacitor 0603")
-    (attr smd)
-    (fp_text reference C3 (at 0 -1.9) (layer F.SilkS)
-      (effects (font (size 1 1) (thickness 0.15)))
-    )
-    (fp_text value 10uF (at 0.04 1.47) (layer F.Fab)
-      (effects (font (size 1 1) (thickness 0.15)))
-    )
-    (fp_line (start -1.45 -0.75) (end 1.45 -0.75) (layer F.CrtYd) (width 0.05))
-    (fp_line (start -1.45 0.75) (end 1.45 0.75) (layer F.CrtYd) (width 0.05))
-    (fp_line (start -1.45 -0.75) (end -1.45 0.75) (layer F.CrtYd) (width 0.05))
-    (fp_line (start 1.45 -0.75) (end 1.45 0.75) (layer F.CrtYd) (width 0.05))
-    (fp_line (start -0.35 -0.6) (end 0.35 -0.6) (layer F.SilkS) (width 0.15))
-    (fp_line (start 0.35 0.6) (end -0.35 0.6) (layer F.SilkS) (width 0.15))
-    (pad 1 smd rect (at -0.75 0) (size 0.8 0.75) (layers F.Cu F.Paste F.Mask)
-      (net 5 "Net-(C3-Pad1)"))
-    (pad 2 smd rect (at 0.75 0) (size 0.8 0.75) (layers F.Cu F.Paste F.Mask)
-      (net 2 GND))
-    (model Capacitors_SMD.3dshapes/C_0603.wrl
-      (at (xyz 0 0 0))
-      (scale (xyz 1 1 1))
-      (rotate (xyz 0 0 0))
-    )
-  )
-  (module Capacitors_SMD:C_0603 (layer F.Cu)
     (at 166.116 86.65 270)
     (descr "Capacitor SMD 0603, reflow soldering, AVX (see smccp.pdf)")
@@
     )
   )
+  (module Capacitors_SMD:C_0805 (layer F.Cu)
+    (at 158.2 88.2)
+    (descr "Capacitor SMD 0805, reflow soldering, AVX (see smccp.pdf)")
+    (tags "capacitor 0805")
+    (attr smd)
+    (fp_text reference C3 (at 0 -2.1) (layer F.SilkS)
+      (effects (font (size 1 1) (thickness 0.15)))
+    )
+    (fp_text value 10uf (at 0 2.1) (layer F.Fab)
+      (effects (font (size 1 1) (thickness 0.15)))
+    )
+    (fp_line (start -1.8 -1) (end 1.8 -1) (layer F.CrtYd) (width 0.05))
+    (fp_line (start -1.8 1) (end 1.8 1) (layer F.CrtYd) (width 0.05))
+    (fp_line (start -1.8 -1) (end -1.8 1) (layer F.CrtYd) (width 0.05))
+    (fp_line (start 1.8 -1) (end 1.8 1) (layer F.CrtYd) (width 0.05))
+    (fp_line (start 0.5 -0.85) (end -0.5 -0.85) (layer F.SilkS) (width 0.15))
+    (fp_line (start -0.5 0.85) (end 0.5 0.85) (layer F.SilkS) (width 0.15))
+    (pad 1 smd rect (at -1 0) (size 1 1.25) (layers F.Cu F.Paste F.Mask)
+      (net 5 "Net-(C3-Pad1)"))
+    (pad 2 smd rect (at 1 0) (size 1 1.25) (layers F.Cu F.Paste F.Mask)
+      (net 2 GND))
+    (model Capacitors_SMD.3dshapes/C_0805.wrl
+      (at (xyz 0 0 0))
+      (scale (xyz 1 1 1))
+      (rotate (xyz 0 0 0))
+    )
+  )
   (gr_text "pyfi, llc\nandy@pyfi.org" (at 202.35 76.2) (layer B.SilkS)
     (effects (font (size 1.5 1.5) (thickness 0.3)) (justify left mirror))
@@
   (segment (start 132.636 66.604) (end 132.636 66.809) (width 0.25) (layer F.Cu) (net 1))
   (segment (start 130.294 64.262) (end 132.636 66.604) (width 0.25) (layer F.Cu) (net 1))
+  (segment (start 159.2 88.2) (end 159.9 88.2) (width 0.25) (layer F.Cu) (net 2))
+  (segment (start 159.9 88.2) (end 160.35 88.65) (width 0.25) (layer F.Cu) (net 2))
+  (via (at 160.35 88.65) (size 0.6) (drill 0.4) (layers F.Cu B.Cu) (net 2))
   (segment (start 159.275 61.15) (end 160.55 61.15) (width 0.25) (layer F.Cu) (net 2))
   (via (at 160.55 61.15) (size 0.6) (drill 0.4) (layers F.Cu B.Cu) (net 2))
@@
   (segment (start 135.00739 70.22461) (end 135.128 70.104) (width 0.25) (layer F.Cu) (net 2))
   (via (at 135.128 70.104) (size 0.6) (drill 0.4) (layers F.Cu B.Cu) (net 2))
-  (segment (start 158.93 88.08) (end 158.93 86.61) (width 0.25) (layer F.Cu) (net 2))
   (segment (start 158.93 86.61) (end 158.82 86.5) (width 0.25) (layer F.Cu) (net 2))
   (segment (start 158.82 85) (end 158.82 86.5) (width 0.25) (layer F.Cu) (net 2))
@@
   (segment (start 162.806 79.56) (end 163.002 79.756) (width 0.25) (layer F.Cu) (net 4))
   (segment (start 156.88 79.56) (end 159.19 79.56) (width 0.25) (layer F.Cu) (net 4))
+  (segment (start 157.2 88.2) (end 157.2 85.12) (width 0.25) (layer F.Cu) (net 5))
+  (segment (start 157.2 85.12) (end 157.32 85) (width 0.25) (layer F.Cu) (net 5))
   (segment (start 163.002 81.026) (end 158.064 81.026) (width 0.25) (layer F.Cu) (net 5))
   (segment (start 157.29 81.8) (end 157.29 82) (width 0.25) (layer F.Cu) (net 5))
@@
   (segment (start 157.29 82.13) (end 157.29 82) (width 0.25) (layer F.Cu) (net 5))
   (segment (start 157.32 85) (end 157.32 82.16) (width 0.25) (layer F.Cu) (net 5))
-  (segment (start 157.43 88.08) (end 157.43 85.11) (width 0.25) (layer F.Cu) (net 5))
   (segment (start 157.43 85.11) (end 157.32 85) (width 0.25) (layer F.Cu) (net 5))
   (segment (start 166.116 85.9) (end 166.902 85.9) (width 0.25) (layer F.Cu) (net 6))
