File: hardware/window-sensor.sch (KiCad schematic (older format))
At the start: 51 parts, among them P1 USB_OTG, Q1 2N7002L, Q2 BSS84LT1G, SW2 SW_PUSH, U1 ESP-WROOM-02, U11 SPX3819, U2 OPA344, U3 CMC-5044PF-A, U4 FT230XS, U5 TSL2581FN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

Commit message: update
Parts:
- R18, R19: Part Number (none) -> ERJ-3GEYJ222V
- R20, R21: Part Number (none) -> ERJ-3EKF1001V
- R5: Part Number (none) -> ERJ-3GEYJ103V
- U1: Part Number (none) -> ESP-WROOM-02
Changed lines of the file:
@@
 LIBS:Zilog
 LIBS:garage-opener-cache
-LIBS:glass-break-cache
+LIBS:window-sensor-cache
 EELAYER 25 0
 EELAYER END
@@
 U 1 1 56C660C8
 P 3550 5150
-F 0 "MBR120-1" H 3550 5250 50  0000 C CNN
+F 0 "MBR120-1" H 3550 5250 50  0001 C CNN
 F 1 "ZENER" H 3550 5050 50  0000 C CNN
 F 2 "Diodes_SMD:SOD-123" H 3550 5150 50  0001 C CNN
@@
 F 2 "garage-opener:ESP-WROOM-02" H 12450 6800 60  0001 C CNN
 F 3 "http://espressif.com/en/products/hardware/esp-wroom-02/resources" H 12450 6800 60  0001 C CNN
+F 4 "ESP-WROOM-02" H 12450 6800 60  0001 C CNN "Part Number"
 	1    12450 6800
 	1    0    0    -1
@@
 F 2 "Resistors_SMD:R_0603" V 12280 7050 50  0001 C CNN
 F 3 "ERJ-3GEYJ103V" H 12350 7050 50  0001 C CNN
+F 4 "ERJ-3GEYJ103V" V 12350 7050 60  0001 C CNN "Part Number"
 	1    12350 7050
 	1    0    0    -1
@@
 F 2 "Resistors_SMD:R_0603" V 11730 7000 50  0001 C CNN
 F 3 "ERJ-3GEYJ222V" H 11800 7000 50  0001 C CNN
+F 4 "ERJ-3GEYJ222V" V 11800 7000 60  0001 C CNN "Part Number"
 	1    11800 7000
 	1    0    0    1
@@
 F 2 "Resistors_SMD:R_0603" V 11580 7000 50  0001 C CNN
 F 3 "ERJ-3GEYJ222V" H 11650 7000 50  0001 C CNN
+F 4 "ERJ-3GEYJ222V" V 11650 7000 60  0001 C CNN "Part Number"
 	1    11650 7000
 	1    0    0    1
@@
 F 2 "Resistors_SMD:R_0603" V 13930 7250 50  0001 C CNN
 F 3 "ERJ-3EKF1001V" H 14000 7250 50  0001 C CNN
+F 4 "ERJ-3EKF1001V" V 14000 7250 60  0001 C CNN "Part Number"
 	1    14000 7250
 	0    1    1    0
@@
 F 2 "Resistors_SMD:R_0603" V 13930 7950 50  0001 C CNN
 F 3 "ERJ-3EKF1001V" H 14000 7950 50  0001 C CNN
+F 4 "ERJ-3EKF1001V" V 14000 7950 60  0001 C CNN "Part Number"
 	1    14000 7950
 	0    1    1    0
